File: zynq_jtag.kicad_sch (KiCad schematic)
At the start: 0 parts

Commit message: sch-updated
Parts:
- added C300: 100n, Capacitor_SMD:C_0402_1005Metric, symbol Device:C
- added D1: RED, LED_0402_RED, symbol Schematic-Lib-PhilsLab:LED_0402_RED
- added D301, D302, D303: Varistor, symbol Device:Varistor
- added D304: Varistor, Diode_SMD:D_0402_1005Metric, symbol Device:Varistor
- added J300: Digilent HS2 Header, Footprint-Lib-PhilsLab:DIGILENT_HS2, symbol Schematic-Lib-PhilsLab:Digilent_HS2_Header
- added Q300: T2N7002AK, Package_TO_SOT_SMD:SOT-23, symbol Transistor_FET:T2N7002AK
- added R1: 510, Resistor_SMD:R_0402_1005Metric, symbol Device:R
- added R300, R301, R302, R303, R304: 4K7, Resistor_SMD:R_0402_1005Metric, symbol Device:R
- added R305, R306, R307, R308: 22R, Resistor_SMD:R_0402_1005Metric, symbol Device:R
- added U1: XC7Z020-2CLG400I, Package_BGA:Xilinx_CLG400, symbol 2024-11-30_12-42-37:XC7Z020-2CLG400I
Connections:
- new net: D302.2, J300.3 (TDO), R306.2
- new net: D303.2, J300.4 (TCK), R307.2
- new net: D304.2, J300.1 (TMS), R308.2
- new net: D301.2, J300.2 (TDI), R305.2
- new net +3V3: C300.1, J300.6 (VDD), R300.2, R301.1, R302.2, R303.2, R304.2
- new net +5V: R1.2
- new net DONE: R302.1, U1.R11 (DONE_0)
- new net GND: C300.2, D301.1, D302.1, D303.1, D304.1, J300.5 (GND)
- new net LED_PWR_A: D1.A, R1.1
- new net NINIT: R303.1, U1.R10 (INIT_B_0)
- new net NPROGRAM: R304.1, U1.L6 (PROGRAM_B_0)
- new net TCK_0: R307.1, U1.F9 (TCK_0)
- new net TDI_0: R300.1, R305.1, U1.G6 (TDI_0)
- new net TDO_0: R306.1, U1.F6 (TDO_0)
- new net TMS_0: R301.2, R308.1, U1.J6 (TMS_0)

Commit message: sch_zynq_update
Parts:
- added C301, C302, C303, C305, C315: 4u7, Capacitor_SMD:C_0402_1005Metric, symbol Device:C
- added C304, C306, C307, C308, C309, C310, C311, C312, C313, C314, C318, C401, C402, C403, C406, C5: 100n, Capacitor_SMD:C_0402_1005Metric, symbol Device:C
- added D305: PMEG1030EJ, Diode_SMD:D_SOD-323F, symbol Diode:PMEG1030EJ
- added D306, D307: Varistor, symbol Device:Varistor
- added D308, D309: RED, LED_0402_RED, symbol Schematic-Lib-PhilsLab:LED_0402_RED
- added FB300, FB301, FB302: 120R, FB_0402, symbol Schematic-Lib-PhilsLab:FB_0402
- added J301: USB-MICRO-B, easyeda2kicad_foorprint:MICRO-USB-SMD_5P-P0.65-H-M_MICRO-USB-5P, symbol Schematic-Lib-PhilsLab:USB3100-30-A
- added R310, R312, R314, R316, R319: 20K, Resistor_SMD:R_0402_1005Metric, symbol Device:R
- added R311, R313, R315, R318, R321: 1k, Resistor_SMD:R_0402_1005Metric, symbol Device:R
- added R317, R320: DNP_OR, Resistor_SMD:R_0402_1005Metric, symbol Device:R
- added R322, R323: 100k, Resistor_SMD:R_0402_1005Metric, symbol Device:R
- added R324, R325, R326, R328, R402: 12K, Resistor_SMD:R_0402_1005Metric, symbol Device:R
- added R325: 2K49, Resistor_SMD:R_0402_1005Metric, symbol Device:R
- added R329, R330, R331, R332, R333, R334, R335, R338, R420: 22R, Resistor_SMD:R_0402_1005Metric, symbol Device:R
- added R336, R337: 510, Resistor_SMD:R_0402_1005Metric, symbol Device:R
- added R403: 4K7, Resistor_SMD:R_0402_1005Metric, symbol Device:R
- added SW300, SW400: SKRPANE010, SKRPANE010, symbol Schematic-Lib-PhilsLab:SKRPANE010
- added SW301: 219-3LPST, Footprint-Lib-PhilsLab:219-3LPST, symbol Schematic-Lib-PhilsLab:219-3LPST
- added U300: FT2232HL-REEL, Footprint-Lib-PhilsLab:LQFP-64-0.5mm, symbol Schematic-Lib-PhilsLab:FT2232HL-REEL
- added U301: 93LC56BT-I/SN, Footprint-Lib-PhilsLab:SOIC-8, symbol Schematic-Lib-PhilsLab:93LC56BT-I/SN
- added U400: SN74LVC1G07DRLR, Footprint-Lib-PhilsLab:SOT-5, symbol Schematic-Lib-PhilsLab:SN74LVC1G07DRLR
- added X300: 12Mhz-TXC Corp, Footprint-Lib-PhilsLab:XTAL_2520, symbol Schematic-Lib-PhilsLab:ECS-2520MV-130-BN-TR
- added X400: ECS-2520MV-33.3, XTAL_2520, symbol Schematic-Lib-PhilsLab:ECS-2520MV-130-BN-TR
- renumbered D1 to D300, R1 to R309
Connections:
- net +5V is gone; now on net +3V3: R309.2
- net +3V3: now also U1.M6 (CFGBVS_0), C310.1, C311.1, C312.1, C313.1, C314.1, C318.1, C403.1, C406.1, C5.1, FB301.1, FB302.1, R317.2, R320.2, R324.2, R325.2, R326.2, R336.2, R337.2, R403.1, SW301.4, SW301.5, SW301.6, U300.20 (VCCIO), U300.31 (VCCIO), U300.42 (VCCIO), U300.50 (VREGIN), U300.56 (VCCIO), U301.8 (VCC), U400.5 (VCC), X300.1 (EN), X300.4 (VDD), X400.1 (EN), X400.4 (VDD)
- net DONE: now also Q300.1 (G)
- net GND: now also Q300.2 (S), U1.K9 (VP_0), U1.L10 (VN_0), U1.M10 (DXN_0), U1.M9 (DXP_0), C301.2, C302.2, C303.2, C304.2, C305.2, C306.2, C307.2, C308.2, C309.2, C310.2, C311.2, C312.2, C313.2, C314.2, C315.2, C318.2, C402.2, C403.2, C406.2, C5.2, D306.2, D307.2, J301.5 (GND), R311.1, R313.1, R315.1, R318.1, R321.1, R323.2, R328.1, SW300.12, U300.1 (GND), U300.10 (AGND), U300.11 (GND), U300.13 (TEST), U300.15 (GND), U300.25 (GND), U300.35 (GND), U300.47 (GND), U300.5 (GND), U300.51 (GND), U301.5 (VSS), U400.3 (GND), X300.2 (GND), X400.2 (GND)
- net NPROGRAM: now also SW300.34
- net TCK_0: now also R329.1
- net TDI_0: now also R330.1
- net TDO_0: no longer U1.F6 (TDO_0)
- net TMS_0: now also R332.1
- net at D300.K: now also Q300.3 (D)
- net PS_NRST: now reaches U1.B10 (PS_SRST_B_501)
- net PS_NRST: now also C401.1, R402.1, SW400.12
- net PS_NPOR: now reaches U1.C7 (PS_POR_B_500)
- net PS_NPOR: now also C402.1, R333.1, R403.2, U400.4 (Y)
- net PS_CLK_33M333: now reaches U1.E7 (PS_CLK_500)
- net PS_CLK_33M333: now also R420.1
- new net: C401.2, SW400.34
- new net: D309.A, R337.1
- new net: D308.A, R336.1
- new net: R324.1, R325.1, U301.4 (DO)
- new net +1V8: R402.2
- new net +1V8_FTDI: C307.1, C308.1, C309.1, C315.1, U300.12 (VCORE), U300.37 (VCORE), U300.49 (VREGOUT), U300.64 (VCORE)
- new net +5V_USB_B: C301.1, FB300.1, J301.1 (VCC)
- new net CGND: J301.0
- new net CLK_12MHZ: R338.2, X300.3 (OUT)
- new net CLK_33M33: R420.2, X400.3 (OUT)
- new net FLASH_CLK_M4: R319.2
- new net FTDI_EECLK: R326.1, U300.62 (EECLK), U301.2 (CLK)
- new net FTDI_EECS: R325.1, U300.63 (EECS), U301.1 (CS)
- new net FTDI_EEDATA: R325.2, U300.61 (EEDATA), U301.3 (DI)
- new net FTDI_NPOR: R333.2, U300.22 (ADBUS5)
- new net FTDI_NRST: R322.2, R323.1, U300.14 (RESET#)
- new net FTDI_OSCI: R338.1, U300.2 (OSCI)
- new net FTDI_REF: R328.2, U300.6 (REF)
- new net FTDI_RX: R335.2, U300.39 (BDBUS1)
- new net FTDI_RX_LED_K: D308.K, U300.54 (BCBUS3)
- new net FTDI_TCK: R329.2, U300.16 (ADBUS0)
- new net FTDI_TDI: R330.2, U300.17 (ADBUS1)
- new net FTDI_TDO: R331.2, U300.18 (ADBUS2)
- new net FTDI_TMS: R332.2, U300.19 (ADBUS3)
- new net FTDI_TX: R334.2, U300.38 (BDBUS0)
- new net FTDI_TX_LED_K: D309.K, U300.55 (BCBUS4)
- new net FTDI_VPHY: C305.1, C306.1, FB302.2, U300.4 (VPHY)
- new net FTDI_VPLL: C303.1, C304.1, FB301.2, U300.9 (VPLL)
- new net M0: R310.1, R311.2, SW301.1
- new net M1: R312.1, R313.2, SW301.2
- new net M2: R314.1, R315.2, SW301.3
- new net M3: R316.1, R317.1, R318.2
- new net M4: R319.1, R320.1, R321.2
- new net PG_3V3: U400.2 (A)
- new net QSPI_DQ0_M3: R316.2
- new net QSPI_DQ1_M1: R312.2
- new net QSPI_DQ2_M2: R314.2
- new net QSPI_DQ3_M0: R310.2
- new net TD0_0: R331.1, U1.F6 (TDO_0)
- new net UART1_RX: R334.1
- new net UART1_TX_VCFG1: R335.1
- new net USB_FTDI_D_N: D306.1, J301.2 (D-), U300.7 (DM)
- new net USB_FTDI_D_P: D307.1, J301.3 (D+), U300.8 (DP)
- new net VCC: D305.1 (K)
- new net VSUB_FILT: C302.1, D305.2 (A), FB300.2, R322.1
- no-connect marks 0 -> 28
Other:
- note added: "BOOT MODE MIO STRAPPING"
- note added: "DONE_LED"
- note added: "FTDI JTAG Programmer and USB-to-UART"
- note added: "JTAG"
- note added: "PS Clock (33.33 MHz)"
- note added: "PS_NPOR"
- note added: "PS_NRST"
- moved on the sheet: C300, D301, D302, D303, D304, J300, R300, R301, R303, R304, R305, R306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

Commit message: sch updated zynq ddr
Parts:
- added C600, C601, C602, C603: 47n, Capacitor_SMD:C_0402_1005Metric, symbol Device:C
- added C604, C605, C606, C607: 470n, Capacitor_SMD:C_0402_1005Metric, symbol Device:C
- added C608, C609, C610, C611: 4u7, Capacitor_SMD:C_0402_1005Metric, symbol Device:C
- added R600, R626, R627: 100R, Resistor_SMD:R_0402_1005Metric, symbol Device:R
- added R601, R602, R603, R604, R605, R606, R607, R608, R609, R610, R611, R612, R613, R614, R615, R616, R617, R618, R619, R620, R621, R622, R623, R624: 49R9, Resistor_SMD:R_0402_1005Metric, symbol Device:R
- added R625: 4K7, Resistor_SMD:R_0402_1005Metric, symbol Device:R
Connections:
- net GND: now also C600.2, C601.2, C602.2, C603.2, C604.2, C605.2, C606.2, C607.2, C608.2, C609.2, C610.2, C611.2, R625.1, R627.1
- net DDR_DM0: now reaches U1.A1 (PS_DDR_DM0_502)
- net DDR_NRST: now reaches U1.B4 (PS_DDR_DRST_B_502)
- net DDR_NRST: now also R625.2
- net DDRA13: now reaches U1.D4 (PS_DDR_A13_502)
- net DDRA13: now also R622.2
- net DDRA12: now reaches U1.E4 (PS_DDR_A12_502)
- net DDRA12: now also R621.2
- net DDR_DM1: now reaches U1.F1 (PS_DDR_DM1_502)
- net DDRA14: now reaches U1.F4 (PS_DDR_A14_502)
- net DDRA14: now also R623.2
- net DDRA10: now reaches U1.F5 (PS_DDR_A10_502)
- net DDRA10: now also R619.2
- net DDRA11: now reaches U1.G4 (PS_DDR_A11_502)
- net DDRA11: now also R620.2
- net DDR_VRN: now reaches U1.G5 (PS_DDR_VRN_502)
- net DDR_VRN: now also R626.2
- net DDR_VRP: now reaches U1.H5 (PS_DDR_VRP_502)
- net DDR_VRP: now also R627.2
- net PL_B35_IO25: now reaches U1.J15 (IO_25_35)
- net DDRA9: now reaches U1.J4 (PS_DDR_A9_502)
- net DDRA9: now also R618.2
- net DDR_BA2: now reaches U1.J5 (PS_DDR_BA2_502)
- net DDR_BA2: now also R608.2
- net DDRA8: now reaches U1.K1 (PS_DDR_A8_502)
- net DDRA8: now also R617.2
- net DDRA1: now reaches U1.K2 (PS_DDR_A1_502)
- net DDRA1: now also R610.2
- net DDRA3: now reaches U1.K3 (PS_DDR_A3_502)
- net DDRA3: now also R612.2
- net DDRA7: now reaches U1.K4 (PS_DDR_A7_502)
- net DDRA7: now also R616.2
- net DDRA5: now reaches U1.L1 (PS_DDR_A5_502)
- net DDRA5: now also R614.2
- net DDR_CK_P: now reaches U1.L2 (PS_DDR_CKP_502)
- net DDR_CK_P: now also R600.2
- net DDRA6: now reaches U1.L4 (PS_DDR_A6_502)
- net DDRA6: now also R615.2
- net DDR_BA0: now reaches U1.L5 (PS_DDR_BA0_502)
- net DDR_BA0: now also R606.2
- net DDR_CK_N: now reaches U1.M2 (PS_DDR_CKN_502)
- net DDR_CK_N: now also R600.1
- net DDRA2: now reaches U1.M3 (PS_DDR_A2_502)
- net DDRA2: now also R611.2
- net DDRA4: now reaches U1.M4 (PS_DDR_A4_502)
- net DDRA4: now also R613.2
- net DDR_NWE: now reaches U1.M5 (PS_DDR_WE_B_502)
- net DDR_NWE: now also R605.2
- net DDR_NCS: now reaches U1.N1 (PS_DDR_CS_B_502)
- net DDR_NCS: now also R602.2
- net DDRA0: now reaches U1.N2 (PS_DDR_A0_502)
- net DDRA0: now also R609.2
- net DDR_CKE: now reaches U1.N3 (PS_DDR_CKE_502)
- net DDR_CKE: now also R601.2
- net DDR_ODT: now reaches U1.N5 (PS_DDR_ODT_502)
- net DDR_ODT: now also R624.2
- net DDR_NRAS: now reaches U1.P4 (PS_DDR_RAS_B_502)
- net DDR_NRAS: now also R603.2
- net DDR_NCAS: now reaches U1.P5 (PS_DDR_CAS_B_502)
- net DDR_NCAS: now also R604.2
- net DDR_BA1: now reaches U1.R4 (PS_DDR_BA1_502)
- net DDR_BA1: now also R607.2
- net DDR_DM2: now reaches U1.T1 (PS_DDR_DM2_502)
- net DDR_DM3: now reaches U1.Y1 (PS_DDR_DM3_502)
- new net +0V675: C600.1, C601.1, C602.1, C603.1, C604.1, C605.1, C606.1, C607.1, C608.1, C609.1, C610.1, C611.1, R601.1, R602.1, R603.1, R604.1, R605.1, R606.1, R607.1, R608.1, R609.1, R610.1, R611.1, R612.1, R613.1, R614.1, R615.1, R616.1, R617.1, R618.1, R619.1, R620.1, R621.1, R622.1, R623.1, R624.1
- new net +1V35: R626.1
- no-connect marks 28 -> 30

Commit message: sch-eth-usb-updated
Parts:
- D301, D302: footprint (none) -> easyeda2kicad_foorprint:C0402
- D303, D306, D307: footprint (none) -> Diode_SMD:D_0402_1005Metric
- renumbered C5 to C316
Changed lines of the file:
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@@
 			)
 		)
-		(property "Footprint" ""
+		(property "Footprint" "easyeda2kicad_foorprint:C0402"
 			(at 45.212 34.29 90)
 			(effects
@@
 			)
 		)
-		(property "Footprint" ""
+		(property "Footprint" "easyeda2kicad_foorprint:C0402"
 			(at 49.022 34.29 90)
 			(effects
@@
 			)
 		)
-		(property "Footprint" ""
+		(property "Footprint" "Diode_SMD:D_0402_1005Metric"
 			(at 300.482 116.84 90)
 			(effects
@@
 		(on_board yes)
 		(dnp no)
-		(property "Reference" "C5"
+		(property "Reference" "C316"
 			(at 292.1 140.462 0)
 			(effects
@@
 			(project "zynq_soc_board_v1"
 				(path "/068a81e1-1783-4521-9958-788ddeed3b49/23d95bc7-ff84-410f-aa0f-c06bb4392e8f"
-					(reference "C5")
+					(reference "C316")
 					(unit 1)
 				)
@@
 			)
 		)
-		(property "Footprint" ""
+		(property "Footprint" "Diode_SMD:D_0402_1005Metric"
 			(at 306.832 116.84 90)
 			(effects
@@
 			)
 		)
-		(property "Footprint" ""
+		(property "Footprint" "Diode_SMD:D_0402_1005Metric"
 			(at 52.578 59.69 90)
 			(effects

Commit message: all page
Parts:
- removed C401, C402, C403, C406: 100n, Capacitor_SMD:C_0402_1005Metric, symbol Device:C
- removed C600, C601, C602, C603: 47n, Capacitor_SMD:C_0402_1005Metric, symbol Device:C
- removed C604, C605, C606, C607: 470n, Capacitor_SMD:C_0402_1005Metric, symbol Device:C
- removed C608, C609, C610, C611: 4u7, Capacitor_SMD:C_0402_1005Metric, symbol Device:C
- removed R402: 12K, Resistor_SMD:R_0402_1005Metric, symbol Device:R
- removed R403, R625: 4K7, Resistor_SMD:R_0402_1005Metric, symbol Device:R
- removed R420: 22R, Resistor_SMD:R_0402_1005Metric, symbol Device:R
- removed R600, R626, R627: 100R, Resistor_SMD:R_0402_1005Metric, symbol Device:R
- removed R601, R602, R603, R604, R605, R606, R607, R608, R609, R610, R611, R612, R613, R614, R615, R616, R617, R618, R619, R620, R621, R622, R623, R624: 49R9, Resistor_SMD:R_0402_1005Metric, symbol Device:R
- removed SW400: SKRPANE010, SKRPANE010, symbol Schematic-Lib-PhilsLab:SKRPANE010
- removed U1: XC7Z020-2CLG400I, Package_BGA:Xilinx_CLG400, symbol 2024-11-30_12-42-37:XC7Z020-2CLG400I
- removed U400: SN74LVC1G07DRLR, Footprint-Lib-PhilsLab:SOT-5, symbol Schematic-Lib-PhilsLab:SN74LVC1G07DRLR
- removed X400: ECS-2520MV-33.3, XTAL_2520, symbol Schematic-Lib-PhilsLab:ECS-2520MV-130-BN-TR
- added U6: XC7Z020-2CLG400I, zynq_sc7z0x0:CLG400, symbol Zynq_xc7z0x0-x:CMP-0363-00007-3
- renumbered R325 to R327
Connections:
- net TD0_0 is gone; now on net TDO_0: R331.1
- net +3V3: now also U6.M6 (CFGBVS_0)
- net DONE: now also U6.R11 (DONE_0)
- net GND: now also U6.K10 (VREFN_0), U6.K9 (VP_0), U6.L10 (VN_0), U6.L9 (VREFP_0), U6.M10 (DXN_0), U6.M9 (DXP_0)
- net NINIT: now also U6.R10 (INIT_B_0)
- net NPROGRAM: now also U6.L6 (PROGRAM_B_0)
- net TCK_0: now also U6.F9 (TCK_0)
- net TDI_0: now also U6.G6 (TDI_0)
- net TDO_0: now also U6.F6 (TDO_0)
- net TMS_0: now also U6.J6 (TMS_0)
- net JTAG_TD0: now reaches D302.2, J300.3 (TDO), R306.2
- net JTAG_TCK: now reaches D303.2, J300.4 (TCK), R307.2
- net JTAG_TMS: now reaches D304.2, J300.1 (TMS), R308.2
- net JTAG_TDI: now reaches D301.2, J300.2 (TDI), R305.2
- net QSPI_DQ3_M0 renamed QSPI_DQ3_M3
- no-connect marks 30 -> 29
Other:
- note added: "Diff Pair"
- note added: "Zynq Config, JTAG"
- note removed: "PS Clock (33.33 MHz)"
- note removed: "PS_NPOR"
- note removed: "PS_NRST"
- title: (none) -> Zynq Config, JTAG, Debug
- moved on the sheet: R302, R303, R304, R310, R311, R312, R313, R314, R315, R316, R317, R318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

Commit message: sch-to-pcb
Connections:
- net FTDI_TX_LED_A: now reaches D309.A, R337.1
- net FTDI_RX_LED_A: now reaches D308.A, R336.1
- net QSPI_DQ3_M3 renamed QSPI_DQ3_M0
Other:
- moved on the sheet: R300, R301, R336, R337

Commit message: xc7z020-fanout
Parts:
- U6: footprint zynq_sc7z0x0:CLG400 -> Package_BGA:Xilinx_CLG400
Changed lines of the file:
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@@
 			)
 		)
-		(property "Footprint" "zynq_sc7z0x0:CLG400"
+		(property "Footprint" "Package_BGA:Xilinx_CLG400"
 			(at 144.78 58.42 0)
 			(effects
