File: power.kicad_sch (KiCad schematic)
At the start: 6 parts, among them U1 LS1205EVD33, U3 BD3539FVM-TR, U4 SY8003ADFC, U5 SY8003ADFC, U6 SY8003ADFC, U7 SY8003ADFC

Commit message: PDF ADDED
Parts:
- added J1: CON-SOCJ-2155, easyeda2kicad_foorprint:DC-IN-TH_DC005-T20, symbol Schematic-Lib-PhilsLab:CON-SOCJ-2155
- U1: LCSC (none) -> C6653278; LOSC C6653278 -> (none)
- U3: LCSC (none) -> C213437; LOSC C213437 -> (none)
Other:
- moved on the sheet: U1
Changed lines of the file:
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@@
 	(symbol
 		(lib_id "Schematic-Lib-PhilsLab:LS1205EVD33")
-		(at 50.8 52.07 0)
+		(at 68.58 49.53 0)
 		(unit 1)
 		(exclude_from_sim no)
@@
 		(fields_autoplaced yes)
 		(property "Reference" "U1"
-			(at 50.8 27.94 0)
+			(at 68.58 25.4 0)
 			(effects
 				(font
@@
 		)
 		(property "Value" "LS1205EVD33"
-			(at 50.8 31.75 0)
+			(at 68.58 29.21 0)
 			(effects
 				(font
@@
 		)
 		(property "Footprint" "Footprint-Lib-PhilsLab:DFN3x3_10L"
-			(at 50.8 52.07 0)
+			(at 68.58 49.53 0)
 			(effects
 				(font
@@
 		)
 		(property "Datasheet" ""
-			(at 50.8 52.07 0)
+			(at 68.58 49.53 0)
 			(effects
 				(font
@@
 		)
 		(property "Description" "18V, 5A eFuse with Programmable Current Limit and Output Voltage Clamp"
-			(at 50.8 52.07 0)
+			(at 68.58 49.53 0)
 			(effects
 				(font
@@
 		)
 		(property "Manufacturer" "Littelfuse"
-			(at 37.592 75.438 0)
+			(at 55.372 72.898 0)
 			(effects
 				(font
@@
 		)
 		(property "Manufacturer Part Number" "LS1205EVD33"
-			(at 37.592 75.438 0)
-			(effects
-				(font
-					(size 1.8288 1.8288)
-				)
-				(justify left bottom)
-				(hide yes)
-			)
-		)
-		(property "LOSC" " C6653278"
-			(at 50.8 52.07 0)
+			(at 55.372 72.898 0)
+			(effects
+				(font
+					(size 1.8288 1.8288)
+				)
+				(justify left bottom)
+				(hide yes)
+			)
+		)
+		(property "LCSC" " C6653278"
+			(at 68.58 49.53 0)
 			(effects
 				(font
@@
 				(path "/068a81e1-1783-4521-9958-788ddeed3b49/e904f396-2c60-426f-aecf-389e552b5c3a"
 					(reference "U1")
+					(unit 1)
+				)
+			)
+		)
+	)
+	(symbol
+		(lib_id "Schematic-Lib-PhilsLab:CON-SOCJ-2155")
+		(at 25.4 44.45 0)
+		(unit 1)
+		(exclude_from_sim no)
+		(in_bom yes)
+		(on_board yes)
+		(dnp no)
+		(fields_autoplaced yes)
+		(property "Reference" "J1"
+			(at 26.7271 27.94 0)
+			(effects
+				(font
+					(size 1.8288 1.8288)
+				)
+			)
+		)
+		(property "Value" "CON-SOCJ-2155"
+			(at 26.7271 31.75 0)
+			(effects
+				(font
+					(size 1.8288 1.8288)
+				)
+			)
+		)
+		(property "Footprint" "easyeda2kicad_foorprint:DC-IN-TH_DC005-T20"
+			(at 25.4 44.45 0)
+			(effects
+				(font
+					(size 1.27 1.27)
+				)
+				(hide yes)
+			)
+		)
+		(property "Datasheet" ""
+			(at 25.4 44.45 0)
+			(effects
+				(font
+					(size 1.27 1.27)
+				)
+				(hide yes)
+			)
+		)
+		(property "Description" "DC Barrell Jack 2.1mm 30V 2.5A THT"
+			(at 25.4 44.45 0)
+			(effects
+				(font
+					(size 1.27 1.27)
+				)
+				(hide yes)
+			)
+		)
+		(property "Manufacturer" "Gravitech"
+			(at 24.13 50.8 0)
+			(effects
+				(font
+					(size 1.8288 1.8288)
+				)
+				(justify left bottom)
+				(hide yes)
+			)
+		)
+		(property "Manufacturer Part Number" "CON-SOCJ-2155"
+			(at 24.13 50.8 0)
+			(effects
+				(font
+					(size 1.8288 1.8288)
+				)
+				(justify left bottom)
+				(hide yes)
+			)
+		)
+		(property "LCSC" "C111567"
+			(at 25.4 44.45 0)
+			(effects
+				(font
+					(size 1.27 1.27)
+				)
+				(hide yes)
+			)
+		)
+		(pin "1"
+		)
+		(pin "2"
+		)
+		(pin "3"
+		)
+		(instances
+			(project ""
+				(path "/068a81e1-1783-4521-9958-788ddeed3b49/e904f396-2c60-426f-aecf-389e552b5c3a"
+					(reference "J1")
 					(unit 1)
 				)
@@
 			)
 		)
-		(property "LOSC" "C213437"
-			(at 54.61 109.22 0)
-			(effects
+		(property "LCSC" "C213437"
+			(at 54.61 109.22 0)
+			(effects

Commit message: sch-updated
Parts:
- removed U5, U6, U7: SY8003ADFC, Footprint-Lib-PhilsLab:DFN2x2-8, symbol Schematic-Lib-PhilsLab:SY8003ADFC
- added C1, C101, C102, C110, C115: 100n, Capacitor_SMD:C_0402_1005Metric, symbol Device:C
- added C100, C103, C104, C107, C108, C109, C112, C113, C114, C117, C118, C119, C122, C123, C124, C127: 22u, Footprint-Lib-PhilsLab:CAP_0805, symbol Device:C
- added C106, C111, C116, C121: 22p, Capacitor_SMD:C_0402_1005Metric, symbol Device:C
- added C120, C125, C126, C128, C129: 4u7, Capacitor_SMD:C_0402_1005Metric, symbol Device:C
- added C130: 1nf, Capacitor_SMD:C_0402_1005Metric, symbol Device:C
- added D100: PMEG1030EJ, Diode_SMD:D_SOD-323F, symbol Diode:PMEG1030EJ
- added D101: RED, LED_0402_RED, symbol Schematic-Lib-PhilsLab:LED_0402_RED
- added L100, L101, L102, L103: 2uh2, SRP0415, symbol Schematic-Lib-PhilsLab:SRP0415-2R2K
- added Q100: T2N7002AK, Package_TO_SOT_SMD:SOT-23, symbol Transistor_FET:T2N7002AK
- added R100, R126: 100k, Resistor_SMD:R_0402_1005Metric, symbol Device:R
- added R101, R103, R105, R108, R110, R113, R115, R118, R120, R123, R125: 12K, Resistor_SMD:R_0402_1005Metric, symbol Device:R
- added R102: 4K7, Resistor_SMD:R_0402_1005Metric, symbol Device:R
- added R104, R107, R109, R112, R114, R117, R119, R122: 100K, Resistor_SMD:R_0402_1005Metric, symbol Device:R
- added R106: 68K, Resistor_SMD:R_0402_1005Metric, symbol Device:R
- added R111: 200K, Resistor_SMD:R_0402_1005Metric, symbol Device:R
- added R116: 124K, Resistor_SMD:R_0402_1005Metric, symbol Device:R
- added R121: 453K, Resistor_SMD:R_0402_1005Metric, symbol Device:R
- added R124: 510, Resistor_SMD:R_0402_1005Metric, symbol Device:R
- added R127: 1k, Resistor_SMD:R_0402_1005Metric, symbol Device:R
- added R128: 1M, Resistor_SMD:R_0402_1005Metric, symbol Device:R
- added U102, U103, U104: SY8003ADFC, Footprint-Lib-PhilsLab:DFN2x2-8, symbol Schematic-Lib-PhilsLab:SY8003ADFC
- renumbered J1 to J100, U1 to U100, U4 to U101, U3 to U105
Connections:
- net VCC: now reaches U100.1 (IN)
- net VCC: now also U100.2 (IN), U100.3 (IN), C100.1, D100.1 (K), R100.1, R101.2
- net +5V: now reaches U100.10 (OUT)
- net +5V: now also U100.8 (OUT), U100.9 (OUT), U101.3 (IN), U105.6 (VCC), U105.7 (VTT_IN), C103.1, C104.1, C109.1, C114.1, C119.1, C124.1, C126.1, R103.2, R105.1, R108.2, R113.2, R118.2, R124.2, U102.3 (IN), U103.3 (IN), U104.3 (IN)
- net GND: now reaches U100.11 (GND)
- net GND: now also J100.2, J100.3, U101.4 (PGND), U101.8 (SGND), U101.9 (PGND), U105.1 (GND), C1.2, C100.2, C101.2, C102.2, C103.2, C104.2, C109.2, C110.2, C114.2, C115.2, C119.2, C120.2, C124.2, C125.2, C126.2, C127.2, C128.2, C129.2, C130.2, Q100.2 (S), R102.1, R104.1, R107.1, R109.1, R112.1, R114.1, R117.1, R119.1, R122.1, R126.2, R128.2, U102.4 (PGND), U102.8 (SGND), U102.9 (PGND), U103.4 (PGND), U103.8 (SGND), U103.9 (PGND), U104.4 (PGND), U104.8 (SGND), U104.9 (PGND)
- net EFUSE_VCP: now reaches U100.4 (VCP)
- net EFUSE_VCP: now also R101.1
- net EFUSE_ILIM: now reaches U100.5 (ILIM)
- net EFUSE_ILIM: now also R102.2
- net EFUSE_SS: now reaches U100.6 (SS)
- net EFUSE_SS: now also C102.1
- net PWR_EN: now reaches U100.7 (EN)
- net PWR_EN: now also C101.1, R100.2
- net +VDC: now reaches J100.1
- net +VDC: now also D100.2 (A)
- net DDR_VTT_EN: now reaches U105.2 (EN)
- net DDR_VTT_EN: now also R125.1, R126.1
- net +0V675: now reaches U105.3 (VTTS)
- net +0V675: now also U105.4 (VREF), U105.8 (VTT), C127.1, C128.1, C129.1
- net DDR_VTT_VDDQ: now reaches U105.5 (VDDQ)
- net DDR_VTT_VDDQ: now also C125.1, R127.2
- net FB_1V0: now reaches U101.1 (FB)
- net FB_1V0: now also C106.2, R106.1, R107.2
- net PG_1V0: now reaches U101.2 (PG)
- net PG_1V0: now also C1.1, R103.1, R104.2, R110.1
- net SW_1V0: now reaches U101.6 (LX)
- net SW_1V0: now also L100.1
- net EN_1V0: now reaches U101.7 (EN)
- net EN_1V0: now also R105.2
- new net: C117.2, C118.2
- new net: C107.2, C108.2
- new net: C122.2, C123.2
- new net: C112.2, C113.2
- new net: Q100.1 (G), R123.1
- new net +1V0: C106.1, C107.1, C108.1, L100.2, R106.2
- new net +1V35: C116.1, C117.1, C118.1, L102.2, R116.2, R127.1
- new net +1V8: C111.1, C112.1, C113.1, L101.2, R111.2
- new net +3V3: C121.1, C122.1, C123.1, L103.2, R121.2
- new net CGND: C130.1, R128.1
- new net EN_1V35: R115.2, U103.7 (EN)
- new net EN_1V8: R110.2, U102.7 (EN)
- new net EN_3V3: R120.2, U104.7 (EN)
- new net FB_1V35: C116.2, R116.1, R117.2, U103.1 (FB)
- new net FB_1V8: C111.2, R111.1, R112.2, U102.1 (FB)
- new net FB_3V3: C121.2, R121.1, R122.2, U104.1 (FB)
- new net LED_PWR_A: D101.A, R124.1
- new net LED_PWR_K: D101.K, Q100.3 (D)
- new net PG_1V35: C115.1, R113.1, R114.2, R120.1, R125.2, U103.2 (PG)
- new net PG_1V8: C110.1, R108.1, R109.2, R115.1, U102.2 (PG)
- new net PG_3V3: C120.1, R118.1, R119.2, R123.2, U104.2 (PG)
- new net SW_1V35: L102.1, U103.6 (LX)
- new net SW_1V8: L101.1, U102.6 (LX)
- new net SW_3V3: L103.1, U104.6 (LX)
- no-connect marks 0 -> 4
Other:
- note added: "BUCK CONVERTERS"
- note added: "DDR3L VTT Regulator"
- note added: "INPUT POWER & EFUSE"
- title: (none) -> Power
- moved on the sheet: U100, U101, U105

Commit message: sch-updated
Parts:
- C1, C101, C102, C110, C115: Manufacturer Part Number CL05B104KO5NNNC -> CL05B104KO5NNNC
- C100, C103, C104, C107, C108, C109, C112, C113, C114, C117, C118, C119, C122, C123, C124, C127: Manufacturer Part Number CL21A226MAQNNNE -> CL21A226MAQNNNE
- C120, C125, C126, C128, C129: LCSC C23733 -> C23733; Manufacturer Part Number CL05A475MP5NRNC -> CL05A475MP5NRNC
- C130: Manufacturer Part Number 0402B102K500NT -> 0402B102K500NT
- R100: LCSC C25741 -> C25741; Manufacturer Part Number 0402WGF1003TCE -> 0402WGF1003TCE
- R102: LCSC C25900 -> C25900
- R103, R105, R108, R110, R113, R115, R118, R123: LCSC C25752 -> C25752
- R116: LCSC C36777 -> C36777; Manufacturer Part Number 0402WGF1243TCE -> 0402WGF1243TCE
- R128: LCSC C26083 -> C26083; Manufacturer Part Number 0402WGF1004TCE -> 0402WGF1004TCE
Changed lines of the file:
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@@
 	(wire
 		(pts
+			(xy 293.37 201.93) (xy 293.37 203.2)
+		)
+		(stroke
+			(width 0)
+			(type default)
+		)
+	)
+	(wire
+		(pts
 			(xy 180.34 50.8) (xy 195.58 50.8)
 		)
@@
 			)
 		)
-		(property "Manufacturer Part Number" " CL21A226MAQNNNE"
+		(property "Manufacturer Part Number" "CL21A226MAQNNNE"
 			(at 288.29 152.4 0)
 			(effects
@@
 			)
 		)
-		(property "LCSC" " C25752"
+		(property "LCSC" "C25752"
 			(at 182.88 153.67 0)
 			(effects
@@
 			)
 		)
-		(property "LCSC" " C25752"
+		(property "LCSC" "C25752"
 			(at 182.88 93.98 0)
 			(effects
@@
 			)
 		)
-		(property "Manufacturer Part Number" " CL21A226MAQNNNE"
+		(property "Manufacturer Part Number" "CL21A226MAQNNNE"
 			(at 292.1 35.56 0)
 			(effects
@@
 			)
 		)
-		(property "Manufacturer Part Number" " CL21A226MAQNNNE"
+		(property "Manufacturer Part Number" "CL21A226MAQNNNE"
 			(at 287.02 207.01 0)
 			(effects
@@
 			)
 		)
-		(property "Manufacturer Part Number" " CL21A226MAQNNNE"
+		(property "Manufacturer Part Number" "CL21A226MAQNNNE"
 			(at 288.29 92.71 0)
 			(effects
@@
 			)
 		)
-		(property "LCSC" " C23733"
+		(property "LCSC" "C23733"
 			(at 80.01 104.14 0)
 			(effects
@@
 			)
 		)
-		(property "Manufacturer Part Number" " CL05A475MP5NRNC"
+		(property "Manufacturer Part Number" "CL05A475MP5NRNC"
 			(at 80.01 104.14 0)
 			(effects
@@
 			)
 		)
-		(property "LCSC" " C25752"
+		(property "LCSC" "C25752"
 			(at 203.2 157.48 0)
 			(effects
@@
 			)
 		)
-		(property "Manufacturer Part Number" " CL21A226MAQNNNE"
+		(property "Manufacturer Part Number" "CL21A226MAQNNNE"
 			(at 187.96 208.28 0)
 			(effects
@@
 			)
 		)
-		(property "Manufacturer Part Number" " CL21A226MAQNNNE"
+		(property "Manufacturer Part Number" "CL21A226MAQNNNE"
 			(at 115.57 43.18 0)
 			(effects
@@
 			)
 		)
-		(property "LCSC" " C25752"
+		(property "LCSC" "C25752"
 			(at 180.34 36.83 0)
 			(effects
@@
 			)
 		)
-		(property "LCSC" " C25900"
+		(property "LCSC" "C25900"
 			(at 105.41 68.58 0)
 			(effects
@@
 			)
 		)
-		(property "Manufacturer Part Number" " CL21A226MAQNNNE"
+		(property "Manufacturer Part Number" "CL21A226MAQNNNE"
 			(at 189.23 93.98 0)
 			(effects
@@
 			)
 		)
-		(property "Manufacturer Part Number" " 0402B102K500NT"
+		(property "Manufacturer Part Number" "0402B102K500NT"
 			(at 38.1 175.26 0)
 			(effects
@@
 			)
 		)
-		(property "LCSC" " C25752"
+		(property "LCSC" "C25752"
 			(at 181.61 208.28 0)
 			(effects
@@
 			)
 		)
-		(property "LCSC" " C25752"
+		(property "LCSC" "C25752"
 			(at 171.45 222.25 0)
 			(effects
@@
 			)
 		)
-		(property "Manufacturer Part Number" " CL21A226MAQNNNE"
+		(property "Manufacturer Part Number" "CL21A226MAQNNNE"
 			(at 24.13 127 0)
 			(effects
@@
 			)
 		)
-		(property "Manufacturer Part Number" " CL05B104KO5NNNC"
+		(property "Manufacturer Part Number" "CL05B104KO5NNNC"
 			(at 182.88 172.72 0)
 			(effects
@@
 			)
 		)
-		(property "LCSC" " C23733"
+		(property "LCSC" "C23733"
 			(at 54.61 134.62 0)
 			(effects
@@
 			)
 		)
-		(property "Manufacturer Part Number" " CL05A475MP5NRNC"
+		(property "Manufacturer Part Number" "CL05A475MP5NRNC"
 			(at 54.61 134.62 0)
 			(effects
@@
 			)
 		)
-		(property "Manufacturer Part Number" " CL21A226MAQNNNE"
+		(property "Manufacturer Part Number" "CL21A226MAQNNNE"
 			(at 189.23 153.67 0)
 			(effects
@@
 			)
 		)
-		(property "LCSC" " C36777"
+		(property "LCSC" "C36777"
 			(at 265.43 153.67 0)
 			(effects
@@
 			)
 		)
-		(property "Manufacturer Part Number" " 0402WGF1243TCE"
+		(property "Manufacturer Part Number" "0402WGF1243TCE"
 			(at 265.43 153.67 0)
 			(effects
@@
 			)
 		)
-		(property "Manufacturer Part Number" " CL21A226MAQNNNE"
+		(property "Manufacturer Part Number" "CL21A226MAQNNNE"
 			(at 294.64 92.71 0)
 			(effects
@@
 			)
 		)
-		(property "Manufacturer Part Number" " CL21A226MAQNNNE"
+		(property "Manufacturer Part Number" "CL21A226MAQNNNE"
 			(at 293.37 207.01 0)
 			(effects
@@
 			)
 		)
-		(property "LCSC" " C26083"
+		(property "LCSC" "C26083"
 			(at 38.1 166.37 0)
 			(effects
@@
 			)
 		)
-		(property "Manufacturer Part Number" " 0402WGF1004TCE"
+		(property "Manufacturer Part Number" "0402WGF1004TCE"
 			(at 38.1 166.37 0)
 			(effects
@@
 			)
 		)
-		(property "LCSC" " C25741"
+		(property "LCSC" "C25741"
 			(at 63.5 43.18 0)
 			(effects
@@
 			)
 		)
-		(property "Manufacturer Part Number" " 0402WGF1003TCE"
+		(property "Manufacturer Part Number" "0402WGF1003TCE"
 			(at 63.5 43.18 0)
 			(effects
@@
 			)
 		)
-		(property "Manufacturer Part Number" " CL05B104KO5NNNC"
+		(property "Manufacturer Part Number" "CL05B104KO5NNNC"
 			(at 68.58 68.58 0)
 			(effects
@@
 	(symbol
 		(lib_id "power:+1V0")
-		(at 293.37 203.2 0)
+		(at 293.37 201.93 0)
 		(unit 1)
 		(exclude_from_sim no)
@@
 		(fields_autoplaced yes)
 		(property "Reference" "#PWR026"
-			(at 293.37 207.01 0)
+			(at 293.37 205.74 0)
 			(effects
 				(font
@@
 		)
 		(property "Value" "+3V3"
-			(at 293.37 198.12 0)
+			(at 293.37 196.85 0)
 			(effects
 				(font
@@
 		)
 		(property "Footprint" ""
-			(at 293.37 203.2 0)
+			(at 293.37 201.93 0)
 			(effects
 				(font
@@
 		)
 		(property "Datasheet" ""
-			(at 293.37 203.2 0)
+			(at 293.37 201.93 0)
 			(effects
 				(font
@@
 		)
 		(property "Description" "Power symbol creates a global label with name \"+1V0\""
-			(at 293.37 203.2 0)
+			(at 293.37 201.93 0)
 			(effects
 				(font
@@
 			)
 		)
-		(property "Manufacturer Part Number" " CL21A226MAQNNNE"
+		(property "Manufacturer Part Number" "CL21A226MAQNNNE"
 			(at 294.64 152.4 0)
 			(effects
@@
 			)
 		)
-		(property "Manufacturer Part Number" " CL05B104KO5NNNC"
+		(property "Manufacturer Part Number" "CL05B104KO5NNNC"
 			(at 182.88 113.03 0)
 			(effects
@@
 			)
 		)
-		(property "LCSC" " C23733"
+		(property "LCSC" "C23733"
 			(at 91.44 134.62 0)
 			(effects
@@
 			)
 		)
-		(property "Manufacturer Part Number" " CL05A475MP5NRNC"
+		(property "Manufacturer Part Number" "CL05A475MP5NRNC"
 			(at 91.44 134.62 0)
 			(effects
@@
 			)
 		)
-		(property "LCSC" " C25752"
+		(property "LCSC" "C25752"
 			(at 203.2 97.79 0)
 			(effects
@@
 			)
 		)
-		(property "Manufacturer Part Number" " CL05B104KO5NNNC"
+		(property "Manufacturer Part Number" "CL05B104KO5NNNC"
 			(at 63.5 68.58 0)
 			(effects
@@
 			)
 		)
-		(property "Manufacturer Part Number" " CL21A226MAQNNNE"
+		(property "Manufacturer Part Number" "CL21A226MAQNNNE"
 			(at 285.75 35.56 0)
 			(effects
@@
 			)
 		)
-		(property "LCSC" " C23733"
+		(property "LCSC" "C23733"
 			(at 181.61 227.33 0)
 			(effects
@@
 			)
 		)
-		(property "Manufacturer Part Number" " CL05A475MP5NRNC"
+		(property "Manufacturer Part Number" "CL05A475MP5NRNC"
 			(at 181.61 227.33 0)
 			(effects
@@
 			)
 		)
-		(property "Manufacturer Part Number" " CL21A226MAQNNNE"
+		(property "Manufacturer Part Number" "CL21A226MAQNNNE"
 			(at 186.69 36.83 0)
 			(effects
@@
 			)
 		)
-		(property "Manufacturer Part Number" " CL05B104KO5NNNC"
+		(property "Manufacturer Part Number" "CL05B104KO5NNNC"
 			(at 180.34 55.88 0)
 			(effects
@@
 			)
 		)
-		(property "Manufacturer Part Number" " CL21A226MAQNNNE"
+		(property "Manufacturer Part Number" "CL21A226MAQNNNE"
 			(at 101.6 118.11 0)
 			(effects
@@
 			)
 		)
-		(property "Manufacturer Part Number" " CL21A226MAQNNNE"
+		(property "Manufacturer Part Number" "CL21A226MAQNNNE"
 			(at 55.88 43.18 0)
 			(effects
@@
 			)
 		)
-		(property "LCSC" " C23733"
+		(property "LCSC" "C23733"
 			(at 107.95 118.11 0)
 			(effects
@@
 			)
 		)
-		(property "Manufacturer Part Number" " CL05A475MP5NRNC"
+		(property "Manufacturer Part Number" "CL05A475MP5NRNC"
 			(at 107.95 118.11 0)
 			(effects
@@
 			)
 		)
-		(property "LCSC" " C25752"
+		(property "LCSC" "C25752"
 			(at 200.66 40.64 0)
 			(effects

Commit message: sch_zynq_update
Parts:
- R101, R120, R125: LCSC C25752 -> C25752
- R126: LCSC C25741 -> C25741; Manufacturer Part Number 0402WGF1003TCE -> 0402WGF1003TCE
- R127: LCSC C11702 -> C11702; Manufacturer Part Number 0402WGF1001TCE -> 0402WGF1001TCE
Changed lines of the file:
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@@
 			)
 		)
-		(property "LCSC" " C25752"
+		(property "LCSC" "C25752"
 			(at 201.93 212.09 0)
 			(effects
@@
 			)
 		)
-		(property "LCSC" " C25752"
+		(property "LCSC" "C25752"
 			(at 107.95 54.61 0)
 			(effects
@@
 			)
 		)
-		(property "LCSC" " C25752"
+		(property "LCSC" "C25752"
 			(at 36.83 107.95 0)
 			(effects
@@
 			)
 		)
-		(property "LCSC" " C11702"
+		(property "LCSC" "C11702"
 			(at 49.53 129.54 0)
 			(effects
@@
 			)
 		)
-		(property "Manufacturer Part Number" " 0402WGF1001TCE"
+		(property "Manufacturer Part Number" "0402WGF1001TCE"
 			(at 49.53 129.54 0)
 			(effects
@@
 			)
 		)
-		(property "LCSC" " C25741"
+		(property "LCSC" "C25741"
 			(at 36.83 127 0)
 			(effects
@@
 			)
 		)
-		(property "Manufacturer Part Number" " 0402WGF1003TCE"
+		(property "Manufacturer Part Number" "0402WGF1003TCE"
 			(at 36.83 127 0)
 			(effects

Commit message: all page
Other:
- note added: "CHASIS GND CONNECTION"
Changed lines of the file:
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@@
+		)
+	)
+	(text "CHASIS GND CONNECTION"
+		(exclude_from_sim no)
+		(at 45.72 161.036 0)
+		(effects
+			(font
+				(size 2.54 2.54)
+				(thickness 0.254)
+				(bold yes)
+			)
 		)
 	)
@@
 				(thickness 0.254)
 				(bold yes)
-			)
-			(justify left bottom)
-		)
-	)
-	(label "CHASIS GND CONNECTION"
-		(at 24.13 161.29 0)
-		(fields_autoplaced yes)
-		(effects
-			(font
-				(size 1.27 1.27)
-				(thickness 0.254)
-				(bold yes)

Commit message: sch-to-pcb
Parts:
- C130: value 1nf -> 1nf,250v; footprint Capacitor_SMD:C_0402_1005Metric -> easyeda2kicad_foorprint:C2211; LCSC C1523 -> C91599; Manufacturer Part Number 0402B102K500NT -> GA352QR7GF102KW01L
- R128: value 1M -> DNP_1M; LCSC C26083 -> (none); Manufacturer Part Number 0402WGF1004TCE -> (none)
Connections:
- net +0V675: no longer C129.1, U105.4 (VREF)
- new net +0V675_REF: C129.1, U105.4 (VREF)

Commit message: xc7z020-fanout
Parts:
- added H1, H2, H3, H4: MountingHole, MountingHole:MountingHole_3.2mm_M3, symbol Mechanical:MountingHole

Commit message: ram-update
Parts:
- D101: footprint LED_0402_RED -> Footprint-Lib-PhilsLab:LED_0402_RED
- L100, L101, L102, L103: footprint SRP0415 -> Footprint-Lib-PhilsLab:SRP0415
- renumbered C1 to C105
Changed lines of the file:
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@@
 			)
 		)
-		(property "Footprint" "SRP0415"
+		(property "Footprint" "Footprint-Lib-PhilsLab:SRP0415"
 			(at 259.08 147.32 0)
 			(effects
@@
 			)
 		)
-		(property "Footprint" "SRP0415"
+		(property "Footprint" "Footprint-Lib-PhilsLab:SRP0415"
 			(at 254 30.48 0)
 			(effects
@@
 			)
 		)
-		(property "Footprint" "LED_0402_RED"
+		(property "Footprint" "Footprint-Lib-PhilsLab:LED_0402_RED"
 			(at 154.94 208.28 0)
 			(effects
@@
 			)
 		)
-		(property "Footprint" "SRP0415"
+		(property "Footprint" "Footprint-Lib-PhilsLab:SRP0415"
 			(at 255.27 201.93 0)
 			(effects
@@
 			)
 		)
-		(property "Footprint" "SRP0415"
+		(property "Footprint" "Footprint-Lib-PhilsLab:SRP0415"
 			(at 257.81 87.63 0)
 			(effects
@@
 		(on_board yes)
 		(dnp no)
-		(property "Reference" "C1"
+		(property "Reference" "C105"
 			(at 175.26 54.102 0)
 			(effects
@@
 			(project "zynq_soc_board_v1"
 				(path "/068a81e1-1783-4521-9958-788ddeed3b49/e904f396-2c60-426f-aecf-389e552b5c3a"
-					(reference "C1")
+					(reference "C105")
 					(unit 1)
 				)
