File: power.kicad_sch (KiCad schematic)
At the start: 78 parts, among them J100 CON-SOCJ-2155, Q100 T2N7002AK, U100 LS1205EVD33, U101 SY8003ADFC, U102 SY8003ADFC, U103 SY8003ADFC, U104 SY8003ADFC, U105 BD3539FVM-TR

Commit message: ram-zynq-updated
Changed lines of the file:
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@@
+	(wire
+		(pts
+			(xy 292.1 29.21) (xy 292.1 31.75)
+		)
+		(stroke
+			(width 0)
+			(type default)
+		)
+	)
 	(wire
 		(pts
@@
 	(symbol
 		(lib_id "power:+1V0")
-		(at 292.1 31.75 0)
+		(at 292.1 29.21 0)
 		(unit 1)
 		(exclude_from_sim no)
@@
 		(fields_autoplaced yes)
 		(property "Reference" "#PWR017"
-			(at 292.1 35.56 0)
+			(at 292.1 33.02 0)
 			(effects
 				(font
@@
 		)
 		(property "Value" "+1V0"
-			(at 292.1 26.67 0)
+			(at 292.1 24.13 0)
 			(effects
 				(font
@@
 		)
 		(property "Footprint" ""
-			(at 292.1 31.75 0)
+			(at 292.1 29.21 0)
 			(effects
 				(font
@@
 		)
 		(property "Datasheet" ""
-			(at 292.1 31.75 0)
+			(at 292.1 29.21 0)
 			(effects
 				(font
@@
 		)
 		(property "Description" "Power symbol creates a global label with name \"+1V0\""
-			(at 292.1 31.75 0)
-			(effects
-				(font
+			(at 292.1 29.21 0)
+			(effects
+				(font

Commit message: pcb_eth
Parts:
- C100, C103, C104, C107, C108, C109, C112, C113, C114, C117, C118, C119, C122, C123, C124, C127: footprint Footprint-Lib-PhilsLab:CAP_0805 -> easyeda2kicad_foorprint:C0805
- L100, L101, L102, L103: footprint Footprint-Lib-PhilsLab:SRP0415 -> easyeda2kicad_foorprint:IND-SMD_L4.4-W4.1
- U101, U102, U103, U104: footprint Footprint-Lib-PhilsLab:DFN2x2-8 -> easyeda2kicad_foorprint:DFN-8_L2.0-W2.0-P0.50-LS2.0-BL-EP
Connections:
- net GND: now also C107.2, C108.2, C112.2, C113.2, C117.2, C118.2, C122.2, C123.2
Changed lines of the file:
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@@
 	)
 	(junction
+		(at 294.64 96.52)
+		(diameter 0)
+		(color 0 0 0 0)
+	)
+	(junction
 		(at 63.5 54.61)
 		(diameter 0)
@@
 	)
 	(junction
+		(at 262.89 60.96)
+		(diameter 0)
+		(color 0 0 0 0)
+	)
+	(junction
 		(at 181.61 201.93)
 		(diameter 0)
@@
 	)
 	(junction
+		(at 293.37 210.82)
+		(diameter 0)
+		(color 0 0 0 0)
+	)
+	(junction
 		(at 222.25 60.96)
 		(diameter 0)
@@
 	)
 	(junction
+		(at 265.43 118.11)
+		(diameter 0)
+		(color 0 0 0 0)
+	)
+	(junction
 		(at 101.6 39.37)
 		(diameter 0)
@@
 	)
 	(junction
+		(at 294.64 156.21)
+		(diameter 0)
+		(color 0 0 0 0)
+	)
+	(junction
 		(at 36.83 119.38)
 		(diameter 0)
@@
 	)
 	(junction
+		(at 265.43 177.8)
+		(diameter 0)
+		(color 0 0 0 0)
+	)
+	(junction
 		(at 274.32 88.9)
 		(diameter 0)
@@
 	)
 	(junction
+		(at 292.1 39.37)
+		(diameter 0)
+		(color 0 0 0 0)
+	)
+	(junction
 		(at 69.85 39.37)
 		(diameter 0)
@@
 	)
 	(junction
+		(at 264.16 232.41)
+		(diameter 0)
+		(color 0 0 0 0)
+	)
+	(junction
 		(at 87.63 72.39)
 		(diameter 0)
@@
 	(wire
 		(pts
+			(xy 294.64 118.11) (xy 294.64 96.52)
+		)
+		(stroke
+			(width 0)
+			(type default)
+		)
+	)
+	(wire
+		(pts
 			(xy 234.95 175.26) (xy 234.95 177.8)
 		)
@@
 	(wire
 		(pts
+			(xy 264.16 232.41) (xy 293.37 232.41)
+		)
+		(stroke
+			(width 0)
+			(type default)
+		)
+	)
+	(wire
+		(pts
 			(xy 189.23 149.86) (xy 189.23 147.32)
 		)
@@
 	(wire
 		(pts
+			(xy 294.64 177.8) (xy 294.64 156.21)
+		)
+		(stroke
+			(width 0)
+			(type default)
+		)
+	)
+	(wire
+		(pts
 			(xy 26.67 175.26) (xy 26.67 166.37)
 		)
@@
 	(wire
 		(pts
+			(xy 292.1 60.96) (xy 292.1 39.37)
+		)
+		(stroke
+			(width 0)
+			(type default)
+		)
+	)
+	(wire
+		(pts
 			(xy 55.88 27.94) (xy 55.88 39.37)
 		)
@@
 	(wire
 		(pts
+			(xy 262.89 60.96) (xy 292.1 60.96)
+		)
+		(stroke
+			(width 0)
+			(type default)
+		)
+	)
+	(wire
+		(pts
 			(xy 196.85 30.48) (xy 209.55 30.48)
 		)
@@
 	(wire
 		(pts
+			(xy 265.43 118.11) (xy 294.64 118.11)
+		)
+		(stroke
+			(width 0)
+			(type default)
+		)
+	)
+	(wire
+		(pts
 			(xy 55.88 46.99) (xy 55.88 73.66)
 		)
@@
 	(wire
 		(pts
+			(xy 265.43 177.8) (xy 294.64 177.8)
+		)
+		(stroke
+			(width 0)
+			(type default)
+		)
+	)
+	(wire
+		(pts
 			(xy 227.33 118.11) (xy 224.79 118.11)
 		)
@@
 	(wire
 		(pts
+			(xy 293.37 232.41) (xy 293.37 210.82)
+		)
+		(stroke
+			(width 0)
+			(type default)
+		)
+	)
+	(wire
+		(pts
 			(xy 189.23 90.17) (xy 189.23 87.63)
 		)
@@
 			)
 		)
-		(property "Footprint" "Footprint-Lib-PhilsLab:CAP_0805"
+		(property "Footprint" "easyeda2kicad_foorprint:C0805"
 			(at 289.2552 156.21 0)
 			(effects
@@
 			)
 		)
-		(property "Footprint" "Footprint-Lib-PhilsLab:CAP_0805"
+		(property "Footprint" "easyeda2kicad_foorprint:C0805"
 			(at 293.0652 39.37 0)
 			(effects
@@
 			)
 		)
-		(property "Footprint" "Footprint-Lib-PhilsLab:CAP_0805"
+		(property "Footprint" "easyeda2kicad_foorprint:C0805"
 			(at 287.9852 210.82 0)
 			(effects
@@
 			)
 		)
-		(property "Footprint" "Footprint-Lib-PhilsLab:DFN2x2-8"
+		(property "Footprint" "easyeda2kicad_foorprint:DFN-8_L2.0-W2.0-P0.50-LS2.0-BL-EP"
 			(at 229.87 97.79 0)
 			(effects
@@
 			)
 		)
-		(property "Footprint" "Footprint-Lib-PhilsLab:SRP0415"
+		(property "Footprint" "easyeda2kicad_foorprint:IND-SMD_L4.4-W4.1"
 			(at 259.08 147.32 0)
 			(effects
@@
 			)
 		)
-		(property "Footprint" "Footprint-Lib-PhilsLab:CAP_0805"
+		(property "Footprint" "easyeda2kicad_foorprint:C0805"
 			(at 289.2552 96.52 0)
 			(effects
@@
 			)
 		)
-		(property "Footprint" "Footprint-Lib-PhilsLab:SRP0415"
+		(property "Footprint" "easyeda2kicad_foorprint:IND-SMD_L4.4-W4.1"
 			(at 254 30.48 0)
 			(effects
@@
 			)
 		)
-		(property "Footprint" "Footprint-Lib-PhilsLab:CAP_0805"
+		(property "Footprint" "easyeda2kicad_foorprint:C0805"
 			(at 188.9252 212.09 0)
 			(effects
@@
 			)
 		)
-		(property "Footprint" "Footprint-Lib-PhilsLab:CAP_0805"
+		(property "Footprint" "easyeda2kicad_foorprint:C0805"
 			(at 116.5352 46.99 0)
 			(effects
@@
 			)
 		)
-		(property "Footprint" "Footprint-Lib-PhilsLab:CAP_0805"
+		(property "Footprint" "easyeda2kicad_foorprint:C0805"
 			(at 190.1952 97.79 0)
 			(effects
@@
 			)
 		)
-		(property "Footprint" "Footprint-Lib-PhilsLab:SRP0415"
+		(property "Footprint" "easyeda2kicad_foorprint:IND-SMD_L4.4-W4.1"
 			(at 255.27 201.93 0)
 			(effects
@@
 			)
 		)
-		(property "Footprint" "Footprint-Lib-PhilsLab:SRP0415"
+		(property "Footprint" "easyeda2kicad_foorprint:IND-SMD_L4.4-W4.1"
 			(at 257.81 87.63 0)
 			(effects
@@
 			)
 		)
-		(property "Footprint" "Footprint-Lib-PhilsLab:CAP_0805"
+		(property "Footprint" "easyeda2kicad_foorprint:C0805"
 			(at 25.0952 130.81 0)
 			(effects
@@
 			)
 		)
-		(property "Footprint" "Footprint-Lib-PhilsLab:DFN2x2-8"
+		(property "Footprint" "easyeda2kicad_foorprint:DFN-8_L2.0-W2.0-P0.50-LS2.0-BL-EP"
 			(at 228.6 212.09 0)
 			(effects
@@
 			)
 		)
-		(property "Footprint" "Footprint-Lib-PhilsLab:CAP_0805"
+		(property "Footprint" "easyeda2kicad_foorprint:C0805"
 			(at 190.1952 157.48 0)
 			(effects
@@
 			)
 		)
-		(property "Footprint" "Footprint-Lib-PhilsLab:CAP_0805"
+		(property "Footprint" "easyeda2kicad_foorprint:C0805"
 			(at 295.6052 96.52 0)
 			(effects
@@
 			)
 		)
-		(property "Footprint" "Footprint-Lib-PhilsLab:CAP_0805"
+		(property "Footprint" "easyeda2kicad_foorprint:C0805"
 			(at 294.3352 210.82 0)
 			(effects
@@
 			)
 		)
-		(property "Footprint" "Footprint-Lib-PhilsLab:CAP_0805"
+		(property "Footprint" "easyeda2kicad_foorprint:C0805"
 			(at 295.6052 156.21 0)
 			(effects
@@
 			)
 		)
-		(property "Footprint" "Footprint-Lib-PhilsLab:DFN2x2-8"
+		(property "Footprint" "easyeda2kicad_foorprint:DFN-8_L2.0-W2.0-P0.50-LS2.0-BL-EP"
 			(at 227.33 40.64 0)
 			(effects
@@
 			)
 		)
-		(property "Footprint" "Footprint-Lib-PhilsLab:CAP_0805"
+		(property "Footprint" "easyeda2kicad_foorprint:C0805"
 			(at 286.7152 39.37 0)
 			(effects
@@
 			)
 		)
-		(property "Footprint" "Footprint-Lib-PhilsLab:CAP_0805"
+		(property "Footprint" "easyeda2kicad_foorprint:C0805"
 			(at 187.6552 40.64 0)
 			(effects
@@
 			)
 		)
-		(property "Footprint" "Footprint-Lib-PhilsLab:CAP_0805"
+		(property "Footprint" "easyeda2kicad_foorprint:C0805"
 			(at 102.5652 121.92 0)
 			(effects
@@
 			)
 		)
-		(property "Footprint" "Footprint-Lib-PhilsLab:DFN2x2-8"
+		(property "Footprint" "easyeda2kicad_foorprint:DFN-8_L2.0-W2.0-P0.50-LS2.0-BL-EP"
 			(at 229.87 157.48 0)
 			(effects
@@
 			)
 		)
-		(property "Footprint" "Footprint-Lib-PhilsLab:CAP_0805"
+		(property "Footprint" "easyeda2kicad_foorprint:C0805"
 			(at 56.8452 46.99 0)
 			(effects

Commit message: usb hs update
Parts:
- R128: footprint Resistor_SMD:R_0402_1005Metric -> Resistor_SMD:R_2010_5025Metric
Changed lines of the file:
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@@
 			)
 		)
-		(property "Footprint" "Resistor_SMD:R_0402_1005Metric"
+		(property "Footprint" "Resistor_SMD:R_2010_5025Metric"
 			(at 38.1 168.148 90)
 			(effects

Commit message: pcb layers
Parts:
- C130: footprint easyeda2kicad_foorprint:C2211 -> Capacitor_SMD:C_1206_3216Metric; LCSC C91599 -> C107211; Manufacturer Part Number GA352QR7GF102KW01L -> CC1206KRX7RYBB102
- D100: footprint Diode_SMD:D_SOD-323F -> easyeda2kicad_foorprint:SOD-323_L1.8-W1.3-LS2.5-RD
- R128: footprint Resistor_SMD:R_2010_5025Metric -> Capacitor_SMD:C_1206_3216Metric
- U100: footprint Footprint-Lib-PhilsLab:DFN3x3_10L -> easyeda2kicad_foorprint:TDFN-10_L3.0-W3.0-P0.50-BL-EP-2.3-1; LCSC C6653278 -> C6653278
- U105: footprint Footprint-Lib-PhilsLab:MSOP8 -> easyeda2kicad_foorprint:MSOP-8_L2.9-W2.8-P0.65-LS4.0-BL
Changed lines of the file:
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@@
 		)
 	)
-	(label "LED_PWR_K"
-		(at 154.94 215.9 0)
-		(fields_autoplaced yes)
-		(effects
-			(font
-				(size 0.508 0.508)
-				(thickness 0.254)
-				(bold yes)
-			)
-			(justify left bottom)
-		)
-	)
 	(label "DDR_VTT_VDDQ"
 		(at 53.34 129.54 0)
@@
 		)
 	)
-	(label "LED_PWR_A"
-		(at 154.94 201.93 0)
-		(fields_autoplaced yes)
-		(effects
-			(font
-				(size 0.508 0.508)
-				(thickness 0.254)
-				(bold yes)
-			)
-			(justify left bottom)
-		)
-	)
 	(label "PG_1V35"
 		(at 203.2 167.64 0)
@@
 		)
 	)
+	(global_label "LED_PWR_A"
+		(shape input)
+		(at 154.94 201.93 180)
+		(fields_autoplaced yes)
+		(effects
+			(font
+				(size 0.762 0.762)
+			)
+			(justify right)
+		)
+		(property "Intersheetrefs" "${INTERSHEET_REFS}"
+			(at 146.8711 201.93 0)
+			(effects
+				(font
+					(size 1.27 1.27)
+				)
+				(justify right)
+				(hide yes)
+			)
+		)
+	)
 	(global_label "PG_1V0"
 		(shape input)
@@
 		)
 	)
+	(global_label "LED_PWR_K"
+		(shape input)
+		(at 154.94 214.63 180)
+		(fields_autoplaced yes)
+		(effects
+			(font
+				(size 0.762 0.762)
+			)
+			(justify right)
+		)
+		(property "Intersheetrefs" "${INTERSHEET_REFS}"
+			(at 146.7622 214.63 0)
+			(effects
+				(font
+					(size 1.27 1.27)
+				)
+				(justify right)
+				(hide yes)
+			)
+		)
+	)
 	(global_label "EFUSE_SS"
 		(shape input)
@@
 			)
 		)
-		(property "Footprint" "Footprint-Lib-PhilsLab:DFN3x3_10L"
+		(property "Footprint" "easyeda2kicad_foorprint:TDFN-10_L3.0-W3.0-P0.50-BL-EP-2.3-1"
 			(at 87.63 52.07 0)
 			(effects
@@
 			)
 		)
-		(property "LCSC" " C6653278"
+		(property "LCSC" "C6653278"
 			(at 87.63 52.07 0)
 			(effects
@@
 			)
 		)
-		(property "Footprint" "Diode_SMD:D_SOD-323F"
+		(property "Footprint" "easyeda2kicad_foorprint:SOD-323_L1.8-W1.3-LS2.5-RD"
 			(at 49.53 34.925 0)
 			(effects
@@
 			)
 		)
-		(property "Footprint" "easyeda2kicad_foorprint:C2211"
+		(property "Footprint" "Capacitor_SMD:C_1206_3216Metric"
 			(at 41.91 174.2948 0)
 			(effects
@@
 			)
 		)
-		(property "LCSC" "C91599"
+		(property "LCSC" "C107211"
 			(at 38.1 175.26 0)
 			(effects
@@
 			)
 		)
-		(property "Manufacturer Part Number" "GA352QR7GF102KW01L"
+		(property "Manufacturer Part Number" "CC1206KRX7RYBB102"
 			(at 38.1 175.26 0)
 			(effects
@@
 			)
 		)
-		(property "Footprint" "Resistor_SMD:R_2010_5025Metric"
+		(property "Footprint" "Capacitor_SMD:C_1206_3216Metric"
 			(at 38.1 168.148 90)
 			(effects
@@
 			)
 		)
-		(property "Footprint" "Footprint-Lib-PhilsLab:MSOP8"
+		(property "Footprint" "easyeda2kicad_foorprint:MSOP-8_L2.9-W2.8-P0.65-LS4.0-BL"
 			(at 73.66 121.92 0)
 			(effects

Commit message: rev a done
Changed lines of the file:
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@@
 	)
 	(junction
+		(at 49.53 212.09)
+		(diameter 0)
+		(color 0 0 0 0)
+	)
+	(junction
 		(at 186.69 30.48)
 		(diameter 0)
@@
 	(wire
 		(pts
+			(xy 41.91 203.2) (xy 41.91 212.09)
+		)
+		(stroke
+			(width 0)
+			(type default)
+		)
+	)
+	(wire
+		(pts
 			(xy 180.34 50.8) (xy 180.34 40.64)
 		)
@@
 	(wire
 		(pts
+			(xy 55.88 203.2) (xy 41.91 203.2)
+		)
+		(stroke
+			(width 0)
+			(type default)
+		)
+	)
+	(wire
+		(pts
 			(xy 271.78 31.75) (xy 262.89 31.75)
 		)
@@
 	(wire
 		(pts
+			(xy 55.88 212.09) (xy 55.88 203.2)
+		)
+		(stroke
+			(width 0)
+			(type default)
+		)
+	)
+	(wire
+		(pts
 			(xy 234.95 175.26) (xy 234.95 177.8)
 		)
@@
 	(wire
 		(pts
+			(xy 49.53 212.09) (xy 49.53 218.44)
+		)
+		(stroke
+			(width 0)
+			(type default)
+		)
+	)
+	(wire
+		(pts
 			(xy 182.88 167.64) (xy 198.12 167.64)
 		)
@@
 	(wire
 		(pts
+			(xy 41.91 212.09) (xy 49.53 212.09)
+		)
+		(stroke
+			(width 0)
+			(type default)
+		)
+	)
+	(wire
+		(pts
 			(xy 189.23 118.11) (xy 201.93 118.11)
 		)
@@
 	(wire
 		(pts
+			(xy 49.53 212.09) (xy 55.88 212.09)
+		)
+		(stroke
+			(width 0)
+			(type default)
+		)
+	)
+	(wire
+		(pts
 			(xy 24.13 123.19) (xy 24.13 114.3)
 		)
@@
 					(unit 1)
 				)
+			)
+		)
+	)
+	(symbol
+		(lib_id "power:Earth")
+		(at 49.53 218.44 0)
+		(unit 1)
+		(exclude_from_sim no)
+		(in_bom yes)
+		(on_board yes)
+		(dnp no)
+		(property "Reference" "#PWR074"
+			(at 49.53 224.79 0)
+			(effects
+				(font
+					(size 1.27 1.27)
+				)
+				(hide yes)
+			)
+		)
+		(property "Value" "CGND"
+			(at 49.53 222.504 0)
+			(effects
+				(font
+					(size 1.27 1.27)
+				)
+			)
+		)
+		(property "Footprint" ""
+			(at 49.53 218.44 0)
+			(effects
+				(font
+					(size 1.27 1.27)
+				)
+				(hide yes)
+			)
+		)
+		(property "Datasheet" "~"
+			(at 49.53 218.44 0)
+			(effects
+				(font
+					(size 1.27 1.27)
+				)
+				(hide yes)
+			)
+		)
+		(property "Description" "Power symbol creates a global label with name \"Earth\""
+			(at 49.53 218.44 0)
+			(effects
+				(font
+					(size 1.27 1.27)
+				)
+				(hide yes)
+			)
+		)
+		(pin "1"
+		)
+		(instances
+			(project "zynq_soc_board_v1"
+				(path "/068a81e1-1783-4521-9958-788ddeed3b49/e904f396-2c60-426f-aecf-389e552b5c3a"
+					(reference "#PWR074")
+					(unit 1)
+				)

Commit message: zynq_soc_complete_hdmi
Changed lines of the file:
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@@
 	(wire
 		(pts
-			(xy 293.37 201.93) (xy 293.37 203.2)
+			(xy 293.37 200.66) (xy 293.37 203.2)
 		)
 		(stroke
@@
 	(symbol
 		(lib_id "power:+1V0")
-		(at 293.37 201.93 0)
+		(at 293.37 200.66 0)
 		(unit 1)
 		(exclude_from_sim no)
@@
 		(fields_autoplaced yes)
 		(property "Reference" "#PWR026"
-			(at 293.37 205.74 0)
+			(at 293.37 204.47 0)
 			(effects
 				(font
@@
 		)
 		(property "Value" "+3V3"
-			(at 293.37 196.85 0)
+			(at 293.37 195.58 0)
 			(effects
 				(font
@@
 		)
 		(property "Footprint" ""
-			(at 293.37 201.93 0)
+			(at 293.37 200.66 0)
 			(effects
 				(font
@@
 		)
 		(property "Datasheet" ""
-			(at 293.37 201.93 0)
+			(at 293.37 200.66 0)
 			(effects
 				(font
@@
 		)
 		(property "Description" "Power symbol creates a global label with name \"+1V0\""
-			(at 293.37 201.93 0)
+			(at 293.37 200.66 0)
 			(effects
 				(font
