File: zynq_processing_system_ps.kicad_sch (KiCad schematic)
At the start: 50 parts, among them Q400 T2N7002AK, SW400 SKRPANE010, U400 SN74LVC1G07DRLR, U401 SN74LVC1G07DRLR, U402 W25Q128JVEIQ, U403 MTFC8GAKAJCN-4M_IT, U6 XC7Z020-2CLG400I, X400 ECS-2520MV-33.3

Commit message: ram-update
Parts:
- D400: footprint LED_0402_RED -> Footprint-Lib-PhilsLab:LED_0402_RED
- R404, R405: footprint Resistor_SMD:R_0402_1005Metric -> easyeda2kicad_foorprint:R0201; LCSC C25765 -> C295787; Manufacturer Part Number 0402WGF2002TCE -> RC0201FR-0720KL
- SW400: footprint SKRPANE010 -> Footprint-Lib-PhilsLab:SKRPANE010
- X400: footprint XTAL_2520 -> Footprint-Lib-PhilsLab:XTAL_2520
Changed lines of the file:
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@@
 			)
 		)
-		(property "Footprint" "XTAL_2520"
+		(property "Footprint" "Footprint-Lib-PhilsLab:XTAL_2520"
 			(at 271.78 214.63 0)
 			(effects
@@
 	)
 	(symbol
-		(lib_id "Device:R")
-		(at 113.03 128.27 270)
-		(unit 1)
-		(exclude_from_sim no)
-		(in_bom yes)
-		(on_board yes)
-		(dnp no)
-		(property "Reference" "R404"
-			(at 113.03 128.27 90)
-			(effects
-				(font
-					(size 0.762 0.762)
-				)
-			)
-		)
-		(property "Value" "20K"
-			(at 109.22 127.508 90)
-			(effects
-				(font
-					(size 0.762 0.762)
-				)
-			)
-		)
-		(property "Footprint" "Resistor_SMD:R_0402_1005Metric"
-			(at 113.03 126.492 90)
-			(effects
-				(font
-					(size 1.27 1.27)
-				)
-				(hide yes)
-			)
-		)
-		(property "Datasheet" "~"
-			(at 113.03 128.27 0)
-			(effects
-				(font
-					(size 1.27 1.27)
-				)
-				(hide yes)
-			)
-		)
-		(property "Description" "Resistor"
-			(at 113.03 128.27 0)
-			(effects
-				(font
-					(size 1.27 1.27)
-				)
-				(hide yes)
-			)
-		)
-		(property "LCSC" "C25765"
-			(at 113.03 128.27 0)
-			(effects
-				(font
-					(size 1.27 1.27)
-				)
-				(hide yes)
-			)
-		)
-		(property "Manufacturer Part Number" "0402WGF2002TCE"
-			(at 113.03 128.27 0)
-			(effects
-				(font
-					(size 1.27 1.27)
-				)
-				(hide yes)
-			)
-		)
-		(pin "2"
-		)
-		(pin "1"
-		)
-		(instances
-			(project "zynq_soc_board_v1"
-				(path "/068a81e1-1783-4521-9958-788ddeed3b49/7169259b-160e-43c7-86a6-e36152f4c13a"
-					(reference "R404")
-					(unit 1)
-				)
-			)
-		)
-	)
-	(symbol
 		(lib_id "Schematic-Lib-PhilsLab:SN74LVC1G07DRLR")
 		(at 157.48 214.63 0)
@@
 			)
 		)
-		(property "Footprint" "SKRPANE010"
+		(property "Footprint" "Footprint-Lib-PhilsLab:SKRPANE010"
 			(at 255.27 60.96 0)
 			(effects
@@
 			)
 		)
-		(property "Footprint" "LED_0402_RED"
+		(property "Footprint" "Footprint-Lib-PhilsLab:LED_0402_RED"
 			(at 195.58 106.68 0)
 			(effects
@@
 	)
 	(symbol
+		(lib_id "Device:R")
+		(at 113.03 128.27 270)
+		(unit 1)
+		(exclude_from_sim no)
+		(in_bom yes)
+		(on_board yes)
+		(dnp no)
+		(property "Reference" "R404"
+			(at 113.03 128.27 90)
+			(effects
+				(font
+					(size 0.762 0.762)
+				)
+			)
+		)
+		(property "Value" "20K"
+			(at 108.712 127.508 90)
+			(effects
+				(font
+					(size 0.762 0.762)
+				)
+			)
+		)
+		(property "Footprint" "easyeda2kicad_foorprint:R0201"
+			(at 113.03 126.492 90)
+			(effects
+				(font
+					(size 1.27 1.27)
+				)
+				(hide yes)
+			)
+		)
+		(property "Datasheet" "~"
+			(at 113.03 128.27 0)
+			(effects
+				(font
+					(size 1.27 1.27)
+				)
+				(hide yes)
+			)
+		)
+		(property "Description" "Resistor"
+			(at 113.03 128.27 0)
+			(effects
+				(font
+					(size 1.27 1.27)
+				)
+				(hide yes)
+			)
+		)
+		(property "LCSC" "C295787"
+			(at 113.03 128.27 0)
+			(effects
+				(font
+					(size 1.27 1.27)
+				)
+				(hide yes)
+			)
+		)
+		(property "Manufacturer Part Number" "RC0201FR-0720KL"
+			(at 113.03 128.27 0)
+			(effects
+				(font
+					(size 1.27 1.27)
+				)
+				(hide yes)
+			)
+		)
+		(pin "2"
+		)
+		(pin "1"
+		)
+		(instances
+			(project "zynq_soc_board_v1"
+				(path "/068a81e1-1783-4521-9958-788ddeed3b49/7169259b-160e-43c7-86a6-e36152f4c13a"
+					(reference "R404")
+					(unit 1)
+				)
+			)
+		)
+	)
+	(symbol
 		(lib_id "power:GND")
 		(at 223.52 62.23 0)
@@
 			)
 		)
-		(property "Footprint" "Resistor_SMD:R_0402_1005Metric"
+		(property "Footprint" "easyeda2kicad_foorprint:R0201"
 			(at 146.05 129.032 90)
 			(effects
@@
 			)
 		)
-		(property "LCSC" "C25765"
+		(property "LCSC" "C295787"
 			(at 146.05 130.81 0)
 			(effects
@@
 			)
 		)
-		(property "Manufacturer Part Number" "0402WGF2002TCE"
+		(property "Manufacturer Part Number" "RC0201FR-0720KL"
 			(at 146.05 130.81 0)
 			(effects
