File: zynq_processing_system_ps.kicad_sch (KiCad schematic)
At the start: 50 parts, among them Q400 T2N7002AK, SW400 SKRPANE010, U400 SN74LVC1G07DRLR, U401 SN74LVC1G07DRLR, U402 W25Q128JVEIQ, U403 MTFC8GAKAJCN-4M_IT, U6 XC7Z020-2CLG400I, X400 ECS-2520MV-33.3

Commit message: pcb_eth
Parts:
- U403: footprint MTFC8GAKAJCN-4M_IT:BGA153N50P14X14_1150X1300X100 -> easyeda2kicad_foorprint:FBGA-153_L13.0-W11.5-P0.50_KLMAG1JETD-B041
Changed lines of the file:
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@@
 			)
 		)
-		(property "Footprint" "MTFC8GAKAJCN-4M_IT:BGA153N50P14X14_1150X1300X100"
+		(property "Footprint" "easyeda2kicad_foorprint:FBGA-153_L13.0-W11.5-P0.50_KLMAG1JETD-B041"
 			(at 339.09 153.67 0)
 			(effects

Commit message: pcb layers
Parts:
- SW400: footprint Footprint-Lib-PhilsLab:SKRPANE010 -> easyeda2kicad_foorprint:SW-SMD_4P-L4.2-W3.2-P2.15-LS4.6-2
- U400, U401: footprint Footprint-Lib-PhilsLab:SOT-5 -> easyeda2kicad_foorprint:SOT-553-5_L1.6-W1.2-P0.50-LS1.6-BL
- U402: footprint Footprint-Lib-PhilsLab:WSON-8-8X6 -> easyeda2kicad_foorprint:WSON-8_L6.0-W8.0-P1.27-BL-EP
- U403: LCSC C395384 -> C395384
Connections:
- net GND: now also C401.2, SW400.34
- net QSPI_NCS: now also R418.2, U402.1 (~{CS})

Commit message: pcbb
Parts:
- SW400: footprint easyeda2kicad_foorprint:SW-SMD_4P-L4.2-W3.2-P2.15-LS4.6-2 -> Footprint-Lib-PhilsLab:SKRPANE010
Changed lines of the file:
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@@
 			)
 		)
-		(property "Footprint" "easyeda2kicad_foorprint:SW-SMD_4P-L4.2-W3.2-P2.15-LS4.6-2"
+		(property "Footprint" "Footprint-Lib-PhilsLab:SKRPANE010"
 			(at 255.27 60.96 0)
 			(effects

Commit message: rev a done
Parts:
- X400: footprint Footprint-Lib-PhilsLab:XTAL_2520 -> Crystal:Crystal_SMD_2520-4Pin_2.5x2.0mm
Changed lines of the file:
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@@
 			)
 		)
-		(property "Footprint" "Footprint-Lib-PhilsLab:XTAL_2520"
+		(property "Footprint" "Crystal:Crystal_SMD_2520-4Pin_2.5x2.0mm"
 			(at 271.78 214.63 0)
 			(effects
