File: zynq_ddr.kicad_sch (KiCad schematic)
At the start: 0 parts

Commit message: sch updated zynq ddr
Parts:
- added C12, C13, C700, C701, C704, C705, C706, C707, C708, C709, C710, C711, C714, C715, C716, C717, C718, C719, C720, C721, C726, C727, C728, C729, C730, C731, C732, C733, C736, C737, C738, C739, C740, C741, C742, C743: 47n, Capacitor_SMD:C_0402_1005Metric, symbol Device:C
- added C702, C712, C724, C734: 4u7, Capacitor_SMD:C_0402_1005Metric, symbol Device:C
- added C703, C713, C725, C735: 470n, Capacitor_SMD:C_0402_1005Metric, symbol Device:C
- added R2, R700: 240R, Resistor_SMD:R_0402_1005Metric, symbol Device:R
- added U3, U5: MT41K256M16TW-107 IT:P, Footprint-Lib-PhilsLab:BGA96C80P9X16_900X1300X120, symbol MT41K256M16TW-107-alt:CMP-2000-06773-2
Connections:
- new net +0V675_REF: C12.2, C13.1, C700.2, C701.1, U3.H1 (VREFDQ), U3.M8 (VREFCA), U5.H1 (VREFDQ), U5.M8 (VREFCA)
- new net +1V35: C12.1, C700.1, C702.1, C703.1, C705.1, C706.1, C707.1, C708.1, C709.1, C710.1, C711.1, C712.1, C713.1, C715.1, C716.1, C717.1, C718.1, C719.1, C720.1, C721.1, C724.1, C725.1, C727.1, C728.1, C729.1, C730.1, C731.1, C732.1, C733.1, C734.1, C735.1, C737.1, C738.1, C739.1, C740.1, C741.1, C742.1, C743.1, U3.A1 (VDDQ), U3.A8 (VDDQ), U3.B2 (VDD), U3.C1 (VDDQ), U3.C9 (VDDQ), U3.D2 (VDDQ), U3.D9 (VDD), U3.E9 (VDDQ), U3.F1 (VDDQ), U3.G7 (VDD), U3.H2 (VDDQ), U3.H9 (VDDQ), U3.K2 (VDD), U3.K8 (VDD), U3.N1 (VDD), U3.N9 (VDD), U3.R1 (VDD), U3.R9 (VDD), U5.A1 (VDDQ), U5.A8 (VDDQ), U5.B2 (VDD), U5.C1 (VDDQ), U5.C9 (VDDQ), U5.D2 (VDDQ), U5.D9 (VDD), U5.E9 (VDDQ), U5.F1 (VDDQ), U5.G7 (VDD), U5.H2 (VDDQ), U5.H9 (VDDQ), U5.K2 (VDD), U5.K8 (VDD), U5.N1 (VDD), U5.N9 (VDD), U5.R1 (VDD), U5.R9 (VDD)
- new net DDR_A0: U3.N3 (A0), U5.N3 (A0)
- new net DDR_A1: U3.P7 (A1), U5.P7 (A1)
- new net DDR_A10: U3.L7 (A10/AP), U5.L7 (A10/AP)
- new net DDR_A11: U3.R7 (A11), U5.R7 (A11)
- new net DDR_A12: U3.N7 (A12/BC#), U5.N7 (A12/BC#)
- new net DDR_A13: U3.T3 (A13), U5.T3 (A13)
- new net DDR_A14: U3.T7 (A14), U5.T7 (A14)
- new net DDR_A2: U3.P3 (A2), U5.P3 (A2)
- new net DDR_A3: U3.N2 (A3), U5.N2 (A3)
- new net DDR_A4: U3.P8 (A4), U5.P8 (A4)
- new net DDR_A5: U3.P2 (A5), U5.P2 (A5)
- new net DDR_A6: U3.R8 (A6), U5.R8 (A6)
- new net DDR_A7: U3.R2 (A7), U5.R2 (A7)
- new net DDR_A8: U3.T8 (A8), U5.T8 (A8)
- new net DDR_A9: U3.R3 (A9), U5.R3 (A9)
- new net DDR_BA0: U3.M2 (BA0), U5.M2 (BA0)
- new net DDR_BA1: U3.N8 (BA1), U5.N8 (BA1)
- new net DDR_BA2: U3.M3 (BA2), U5.M3 (BA2)
- new net DDR_CKE: U3.K9 (CKE), U5.K9 (CKE)
- new net DDR_CK_N: U3.K7 (CK#), U5.K7 (CK#)
- new net DDR_CK_P: U3.J7 (CK), U5.J7 (CK)
- new net DDR_DM0: U3.D3 (UDM)
- new net DDR_DM1: U3.E7 (LDM)
- new net DDR_DM2: U5.E7 (LDM)
- new net DDR_DM3: U5.D3 (UDM)
- new net DDR_DQ0: U3.A3 (DQ15)
- new net DDR_DQ1: U3.C3 (DQ9)
- new net DDR_DQ10: U3.G2 (DQ6)
- new net DDR_DQ11: U3.H7 (DQ7)
- new net DDR_DQ12: U3.F7 (DQ1)
- new net DDR_DQ13: U3.H8 (DQ5)
- new net DDR_DQ14: U3.F2 (DQ2)
- new net DDR_DQ15: U3.F8 (DQ3)
- new net DDR_DQ16: U5.E3 (DQ0)
- new net DDR_DQ17: U5.H3 (DQ4)
- new net DDR_DQ18: U5.G2 (DQ6)
- new net DDR_DQ19: U5.F2 (DQ2)
- new net DDR_DQ2: U3.C2 (DQ11)
- new net DDR_DQ20: U5.F7 (DQ1)
- new net DDR_DQ21: U5.F8 (DQ3)
- new net DDR_DQ22: U5.H8 (DQ5)
- new net DDR_DQ23: U5.H7 (DQ7)
- new net DDR_DQ24: U5.A2 (DQ13)
- new net DDR_DQ25: U5.C8 (DQ10)
- new net DDR_DQ26: U5.A3 (DQ15)
- new net DDR_DQ27: U5.B8 (DQ14)
- new net DDR_DQ28: U5.C3 (DQ9)
- new net DDR_DQ29: U5.D7 (DQ8)
- new net DDR_DQ3: U3.A2 (DQ13)
- new net DDR_DQ30: U5.C2 (DQ11)
- new net DDR_DQ31: U5.A7 (DQ12)
- new net DDR_DQ4: U3.B8 (DQ14)
- new net DDR_DQ5: U3.D7 (DQ8)
- new net DDR_DQ6: U3.A7 (DQ12)
- new net DDR_DQ7: U3.C8 (DQ10)
- new net DDR_DQ8: U3.H3 (DQ4)
- new net DDR_DQ9: U3.E3 (DQ0)
- new net DDR_DQS0_N: U3.B7 (UDQS#)
- new net DDR_DQS0_P: U3.C7 (UDQS)
- new net DDR_DQS1_N: U3.G3 (LDQS#)
- new net DDR_DQS1_P: U3.F3 (LDQS)
- new net DDR_DQS2_N: U5.G3 (LDQS#)
- new net DDR_DQS2_P: U5.F3 (LDQS)
- new net DDR_DQS3_N: U5.B7 (UDQS#)
- new net DDR_DQS3_P: U5.C7 (UDQS)
- new net DDR_NCAS: U3.K3 (CAS#), U5.K3 (CAS#)
- new net DDR_NCS: U3.L2 (CS#), U5.L2 (CS#)
- new net DDR_NRAS: U3.J3 (RAS#), U5.J3 (RAS#)
- new net DDR_NRST: U3.T2 (RESET#), U5.T2 (RESET#)
- new net DDR_NWE: U3.L3 (WE#), U5.L3 (WE#)
- new net DDR_ODT: U3.K1 (ODT), U5.K1 (ODT)
- new net DDR_ZQ1: R700.2, U3.L8 (ZQ)
- new net DDR_ZQ2: R2.2, U5.L8 (ZQ)
- new net GND: C13.2, C701.2, C702.2, C703.2, C705.2, C706.2, C707.2, C708.2, C709.2, C710.2, C711.2, C712.2, C713.2, C715.2, C716.2, C717.2, C718.2, C719.2, C720.2, C721.2, C724.2, C725.2, C727.2, C728.2, C729.2, C730.2, C731.2, C732.2, C733.2, C734.2, C735.2, C737.2, C738.2, C739.2, C740.2, C741.2, C742.2, C743.2, R2.1, R700.1, U3.A9 (VSS), U3.B1 (VSSQ), U3.B3 (VSS), U3.B9 (VSSQ), U3.D1 (VSSQ), U3.D8 (VSSQ), U3.E1 (VSS), U3.E2 (VSSQ), U3.E8 (VSSQ), U3.F9 (VSSQ), U3.G1 (VSSQ), U3.G8 (VSS), U3.G9 (VSSQ), U3.J2 (VSS), U3.J8 (VSS), U3.M1 (VSS), U3.M9 (VSS), U3.P1 (VSS), U3.P9 (VSS), U3.T1 (VSS), U3.T9 (VSS), U5.A9 (VSS), U5.B1 (VSSQ), U5.B3 (VSS), U5.B9 (VSSQ), U5.D1 (VSSQ), U5.D8 (VSSQ), U5.E1 (VSS), U5.E2 (VSSQ), U5.E8 (VSSQ), U5.F9 (VSSQ), U5.G1 (VSSQ), U5.G8 (VSS), U5.G9 (VSSQ), U5.J2 (VSS), U5.J8 (VSS), U5.M1 (VSS), U5.M9 (VSS), U5.P1 (VSS), U5.P9 (VSS), U5.T1 (VSS), U5.T9 (VSS)
- no-connect marks 0 -> 10
Other:
- note added: "ACC & DAT Connection"
- note added: "Power and Decoupling"

Commit message: all page
Parts:
- added C600, C601, C602, C603, C612, C613: 47n, Capacitor_SMD:C_0402_1005Metric, symbol Device:C
- added C604, C605, C606, C607: 470n, Capacitor_SMD:C_0402_1005Metric, symbol Device:C
- added C608, C609, C610, C611: 4u7, Capacitor_SMD:C_0402_1005Metric, symbol Device:C
- added R600, R626, R627: 100R, Resistor_SMD:R_0402_1005Metric, symbol Device:R
- added R601, R602, R603, R604, R605, R606, R607, R608, R609, R610, R611, R612, R613, R614, R615, R616, R617, R618, R619, R620, R621, R622, R623, R624: 49R9, Resistor_SMD:R_0402_1005Metric, symbol Device:R
- added R625: 4K7, Resistor_SMD:R_0402_1005Metric, symbol Device:R
- added U6: XC7Z020-2CLG400I, zynq_sc7z0x0:CLG400, symbol Zynq_xc7z0x0-x:CMP-0363-00007-3
- renumbered R2 to R701, U3 to U700, U5 to U701
Connections:
- net +0V675_REF: now also C612.1, C613.1, U6.H6 (PS_DDR_VREF0_502), U6.P6 (PS_DDR_VREF1_502)
- net +1V35: now also C704.1, C714.1, C726.1, C736.1, R626.1
- net DDR_A0: now also R609.2, U6.N2 (PS_DDR_A0_502)
- net DDR_A1: now also R610.2, U6.K2 (PS_DDR_A1_502)
- net DDR_A10: now also R619.2, U6.F5 (PS_DDR_A10_502)
- net DDR_A11: now also R620.2, U6.G4 (PS_DDR_A11_502)
- net DDR_A12: now also R621.2, U6.E4 (PS_DDR_A12_502)
- net DDR_A13: now also R622.2, U6.D4 (PS_DDR_A13_502)
- net DDR_A14: now also R623.2, U6.F4 (PS_DDR_A14_502)
- net DDR_A2: now also R611.2, U6.M3 (PS_DDR_A2_502)
- net DDR_A3: now also R612.2, U6.K3 (PS_DDR_A3_502)
- net DDR_A4: now also R613.2, U6.M4 (PS_DDR_A4_502)
- net DDR_A5: now also R614.2, U6.L1 (PS_DDR_A5_502)
- net DDR_A6: now also R615.2, U6.L4 (PS_DDR_A6_502)
- net DDR_A7: now also R616.2, U6.K4 (PS_DDR_A7_502)
- net DDR_A8: now also R617.2, U6.K1 (PS_DDR_A8_502)
- net DDR_A9: now also R618.2, U6.J4 (PS_DDR_A9_502)
- net DDR_BA0: now also R606.2, U6.L5 (PS_DDR_BA0_502)
- net DDR_BA1: now also R607.2, U6.R4 (PS_DDR_BA1_502)
- net DDR_BA2: now also R608.2, U6.J5 (PS_DDR_BA2_502)
- net DDR_CKE: now also R601.2, U6.N3 (PS_DDR_CKE_502)
- net DDR_CK_N: now also R600.1, U6.M2 (PS_DDR_CKN_502)
- net DDR_CK_P: now also R600.2, U6.L2 (PS_DDR_CKP_502)
- net DDR_DM0: now also U6.A1 (PS_DDR_DM0_502)
- net DDR_DM1: now also U6.F1 (PS_DDR_DM1_502)
- net DDR_DM2: now also U6.T1 (PS_DDR_DM2_502)
- net DDR_DM3: now also U6.Y1 (PS_DDR_DM3_502)
- net DDR_DQ0: now also U6.C3 (PS_DDR_DQ0_502)
- net DDR_DQ1: now also U6.B3 (PS_DDR_DQ1_502)
- net DDR_DQ10: now also U6.G3 (PS_DDR_DQ10_502)
- net DDR_DQ11: now also U6.H3 (PS_DDR_DQ11_502)
- net DDR_DQ12: now also U6.J3 (PS_DDR_DQ12_502)
- net DDR_DQ13: now also U6.H2 (PS_DDR_DQ13_502)
- net DDR_DQ14: now also U6.H1 (PS_DDR_DQ14_502)
- net DDR_DQ15: now also U6.J1 (PS_DDR_DQ15_502)
- net DDR_DQ16: now also U6.P1 (PS_DDR_DQ16_502)
- net DDR_DQ17: now also U6.P3 (PS_DDR_DQ17_502)
- net DDR_DQ18: now also U6.R3 (PS_DDR_DQ18_502)
- net DDR_DQ19: now also U6.R1 (PS_DDR_DQ19_502)
- net DDR_DQ2: now also U6.A2 (PS_DDR_DQ2_502)
- net DDR_DQ20: now also U6.T4 (PS_DDR_DQ20_502)
- net DDR_DQ21: now also U6.U4 (PS_DDR_DQ21_502)
- net DDR_DQ22: now also U6.U2 (PS_DDR_DQ22_502)
- net DDR_DQ23: now also U6.U3 (PS_DDR_DQ23_502)
- net DDR_DQ24: now also U6.V1 (PS_DDR_DQ24_502)
- net DDR_DQ25: now also U6.Y3 (PS_DDR_DQ25_502)
- net DDR_DQ26: now also U6.W1 (PS_DDR_DQ26_502)
- net DDR_DQ27: now also U6.Y4 (PS_DDR_DQ27_502)
- net DDR_DQ28: now also U6.Y2 (PS_DDR_DQ28_502)
- net DDR_DQ29: now also U6.W3 (PS_DDR_DQ29_502)
- net DDR_DQ3: now also U6.A4 (PS_DDR_DQ3_502)
- net DDR_DQ30: now also U6.V2 (PS_DDR_DQ30_502)
- net DDR_DQ31: now also U6.V3 (PS_DDR_DQ31_502)
- net DDR_DQ4: now also U6.D3 (PS_DDR_DQ4_502)
- net DDR_DQ5: now also U6.D1 (PS_DDR_DQ5_502)
- net DDR_DQ6: now also U6.C1 (PS_DDR_DQ6_502)
- net DDR_DQ7: now also U6.E1 (PS_DDR_DQ7_502)
- net DDR_DQ8: now also U6.E2 (PS_DDR_DQ8_502)
- net DDR_DQ9: now also U6.E3 (PS_DDR_DQ9_502)
- net DDR_DQS0_N: now also U6.B2 (PS_DDR_DQS_N0_502)
- net DDR_DQS0_P: now also U6.C2 (PS_DDR_DQS_P0_502)
- net DDR_DQS1_N: now also U6.F2 (PS_DDR_DQS_N1_502)
- net DDR_DQS1_P: now also U6.G2 (PS_DDR_DQS_P1_502)
- net DDR_DQS2_N: now also U6.T2 (PS_DDR_DQS_N2_502)
- net DDR_DQS2_P: now also U6.R2 (PS_DDR_DQS_P2_502)
- net DDR_DQS3_N: now also U6.W4 (PS_DDR_DQS_N3_502)
- net DDR_DQS3_P: now also U6.W5 (PS_DDR_DQS_P3_502)
- net DDR_NCAS: now also R604.2, U6.P5 (PS_DDR_CAS_B_502)
- net DDR_NCS: now also R602.2, U6.N1 (PS_DDR_CS_B_502)
- net DDR_NRAS: now also R603.2, U6.P4 (PS_DDR_RAS_B_502)
- net DDR_NRST: now also R625.2, U6.B4 (PS_DDR_DRST_B_502)
- net DDR_NWE: now also R605.2, U6.M5 (PS_DDR_WE_B_502)
- net DDR_ODT: now also R624.2, U6.N5 (PS_DDR_ODT_502)
- net GND: now also C704.2, C714.2, C726.2, C736.2, C600.2, C601.2, C602.2, C603.2, C604.2, C605.2, C606.2, C607.2, C608.2, C609.2, C610.2, C611.2, C612.2, C613.2, R625.1, R627.2
- new net +0V675: C600.1, C601.1, C602.1, C603.1, C604.1, C605.1, C606.1, C607.1, C608.1, C609.1, C610.1, C611.1, R601.1, R602.1, R603.1, R604.1, R605.1, R606.1, R607.1, R608.1, R609.1, R610.1, R611.1, R612.1, R613.1, R614.1, R615.1, R616.1, R617.1, R618.1, R619.1, R620.1, R621.1, R622.1, R623.1, R624.1
- new net DDR_VRN: R626.2, U6.G5 (PS_DDR_VRN_502)
- new net DDR_VRP: R627.1, U6.H5 (PS_DDR_VRP_502)
Other:
- note added: "Diff Pair"
- note added: "Zynq DDR Interface"
- title: (none) -> Zynq DDR Interface & 1GB DDR3L Modules
- moved on the sheet: C12, C13, C700, C701, C702, C703, C704, C705, C706, C707, C708, C709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

Commit message: sch-to-pcb
Other:
- moved on the sheet: C716
Changed lines of the file:
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@@
 	)
 	(junction
+		(at 139.7 86.36)
+		(diameter 0)
+		(color 0 0 0 0)
+	)
+	(junction
 		(at 153.1379 156.21)
 		(diameter 0)
@@
 	)
 	(junction
-		(at 139.1679 78.74)
-		(diameter 0)
-		(color 0 0 0 0)
-	)
-	(junction
 		(at 212.09 40.64)
 		(diameter 0)
@@
 	)
 	(junction
-		(at 139.1679 86.36)
-		(diameter 0)
-		(color 0 0 0 0)
-	)
-	(junction
 		(at 373.38 102.87)
 		(diameter 0)
@@
 	)
 	(junction
+		(at 139.7 78.74)
+		(diameter 0)
+		(color 0 0 0 0)
+	)
+	(junction
 		(at 165.1 60.96)
 		(diameter 0)
@@
 	(wire
 		(pts
+			(xy 139.7 78.74) (xy 146.05 78.74)
+		)
+		(stroke
+			(width 0)
+			(type default)
+		)
+	)
+	(wire
+		(pts
 			(xy 339.09 184.15) (xy 377.19 184.15)
 		)
@@
 	(wire
 		(pts
-			(xy 139.1679 78.74) (xy 146.05 78.74)
-		)
-		(stroke
-			(width 0)
-			(type default)
-		)
-	)
-	(wire
-		(pts
 			(xy 179.07 76.2) (xy 180.34 76.2)
 		)
@@
 	(wire
 		(pts
-			(xy 132.08 86.36) (xy 139.1679 86.36)
+			(xy 132.08 86.36) (xy 139.7 86.36)
 		)
 		(stroke
@@
 	(wire
 		(pts
-			(xy 139.1679 86.36) (xy 146.05 86.36)
-		)
-		(stroke
-			(width 0)
-			(type default)
-		)
-	)
-	(wire
-		(pts
 			(xy 373.38 133.35) (xy 373.38 135.89)
 		)
@@
 	(wire
 		(pts
+			(xy 139.7 86.36) (xy 146.05 86.36)
+		)
+		(stroke
+			(width 0)
+			(type default)
+		)
+	)
+	(wire
+		(pts
 			(xy 80.01 177.8) (xy 95.25 177.8)
 		)
@@
 	(wire
 		(pts
-			(xy 132.08 78.74) (xy 139.1679 78.74)
+			(xy 132.08 78.74) (xy 139.7 78.74)
 		)
 		(stroke
@@
 	(symbol
 		(lib_id "Device:C")
-		(at 139.1679 82.55 0)
+		(at 139.7 82.55 0)
 		(unit 1)
 		(exclude_from_sim no)
@@
 		(dnp no)
 		(property "Reference" "C716"
-			(at 139.1679 80.772 0)
+			(at 139.7 80.772 0)
 			(effects
 				(font
@@
 		)
 		(property "Value" "47n"
-			(at 139.1679 84.582 0)
+			(at 139.7 84.582 0)
 			(effects
 				(font
@@
 		)
 		(property "Footprint" "Capacitor_SMD:C_0402_1005Metric"
-			(at 140.1331 86.36 0)
+			(at 140.6652 86.36 0)
 			(effects
 				(font
@@
 		)
 		(property "Datasheet" "~"
-			(at 139.1679 82.55 0)
+			(at 139.7 82.55 0)
 			(effects
 				(font
@@
 		)
 		(property "Description" "Unpolarized capacitor"
-			(at 139.1679 82.55 0)
+			(at 139.7 82.55 0)
 			(effects
 				(font
@@
 		)
 		(property "LCSC" "C47339"
-			(at 139.1679 82.55 0)
+			(at 139.7 82.55 0)
 			(effects
 				(font
@@
 		)
 		(property "Manufacturer Part Number" "CL05A474KP5NNNC"
-			(at 139.1679 82.55 0)
+			(at 139.7 82.55 0)
 			(effects
 				(font
@@
 		(dnp no)
 		(property "Reference" "R627"
-			(at 375.412 187.96 90)
+			(at 373.126 187.452 0)
 			(effects
 				(font
@@
 		)
 		(property "Value" "100R"
-			(at 377.19 188.468 90)
+			(at 373.126 189.484 0)
 			(effects
 				(font
@@
 		(dnp no)
 		(property "Reference" "R626"
-			(at 375.412 177.8 90)
+			(at 373.634 175.768 0)
 			(effects
 				(font
@@
 		)
 		(property "Value" "100R"
-			(at 377.19 178.308 90)
+			(at 373.888 177.8 0)
 			(effects
 				(font

Commit message: xc7z020-fanout
Parts:
- U6: footprint zynq_sc7z0x0:CLG400 -> Package_BGA:Xilinx_CLG400
Changed lines of the file:
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@@
 			)
 		)
-		(property "Footprint" "zynq_sc7z0x0:CLG400"
+		(property "Footprint" "Package_BGA:Xilinx_CLG400"
 			(at 280.67 74.93 0)
 			(effects

Commit message: ram-update
Parts:
- removed C12, C13: 47n, Capacitor_SMD:C_0402_1005Metric, symbol Device:C
- added C722, C723: 47n, easyeda2kicad_foorprint:C0201, symbol Device:C
- C600, C601, C602, C603, C612, C613, C700, C701, C704, C705, C706, C707, C708, C709, C710, C711, C714, C715, C716, C717, C718, C719, C720, C721: footprint Capacitor_SMD:C_0402_1005Metric -> easyeda2kicad_foorprint:C0201; LCSC C47339 -> C88917; Manufacturer Part Number CL05A474KP5NNNC -> GRM033R61C473KE84D
- C604, C605, C606, C607, C703, C713: footprint Capacitor_SMD:C_0402_1005Metric -> easyeda2kicad_foorprint:C0201; LCSC C47339 -> C76591; Manufacturer Part Number CL05A474KP5NNNC -> C0603X5R1A474MT00NE
- C712: footprint Capacitor_SMD:C_0402_1005Metric -> easyeda2kicad_foorprint:C0201
- C725, C735: footprint Capacitor_SMD:C_0402_1005Metric -> Capacitor_SMD:C_0201_0603Metric; LCSC C47339 -> C76591; Manufacturer Part Number CL05A474KP5NNNC -> C0603X5R1A474MT00NE
- C726, C727, C728, C729, C730, C731, C732, C733, C736, C737, C738, C739, C740, C741, C742, C743: footprint Capacitor_SMD:C_0402_1005Metric -> Capacitor_SMD:C_0201_0603Metric; LCSC C47339 -> C88917; Manufacturer Part Number CL05A474KP5NNNC -> GRM033R61C473KE84D
- R600, R626, R627: footprint Resistor_SMD:R_0402_1005Metric -> easyeda2kicad_foorprint:R0201; LCSC C25076 -> C77623; Manufacturer Part Number 0402WGF1000TCE -> RC0201FR-07100RL
- R601, R602, R603, R604, R605, R606, R607, R608, R609, R610, R611, R612, R613, R614, R615, R616, R617, R618, R619, R620, R621, R622, R623, R624: footprint Resistor_SMD:R_0402_1005Metric -> easyeda2kicad_foorprint:R0201; LCSC C25120 -> C155744; Manufacturer Part Number 0402WGF499JTCE -> RC0201FR-0749R9L
Connections:
- net +0V675_REF: now also C722.2, C723.1
- net +1V35: now also C722.1
- net GND: now also C723.2

Commit message: ram-zynq-updated
Other:
- note added: "DDR_ACC"
- note added: "DDR_BL0"
- note added: "DDR_BL1"
- note added: "DDR_BL2"
- note added: "DDR_BL3"
