File: zynq_ddr.kicad_sch (KiCad schematic)
At the start: 91 parts, among them U6 XC7Z020-2CLG400I, U700 MT41K256M16TW-107 IT:P, U701 MT41K256M16TW-107 IT:P

Commit message: pcb_eth
Parts:
- U700, U701: footprint Footprint-Lib-PhilsLab:BGA96C80P9X16_900X1300X120 -> easyeda2kicad_foorprint:FBGA-96_L14.0-W8.0-R16-C6-P0.80-TL; LCSC (none) -> C367428; Manufacturer Part Number (none) -> MT41K256M16TW-107 IT:P
Changed lines of the file:
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@@
 			)
 		)
-		(property "Footprint" "Footprint-Lib-PhilsLab:BGA96C80P9X16_900X1300X120"
+		(property "Footprint" "easyeda2kicad_foorprint:FBGA-96_L14.0-W8.0-R16-C6-P0.80-TL"
 			(at 185.42 30.48 0)
 			(effects
@@
 			)
 		)
+		(property "LCSC" "C367428"
+			(at 185.42 30.48 0)
+			(effects
+				(font
+					(size 1.27 1.27)
+				)
+				(hide yes)
+			)
+		)
+		(property "Manufacturer Part Number" "MT41K256M16TW-107 IT:P"
+			(at 185.42 30.48 0)
+			(effects
+				(font
+					(size 1.27 1.27)
+				)
+				(hide yes)
+			)
+		)
 		(pin "J9"
 		)
@@
 			)
 		)
-		(property "Footprint" "Footprint-Lib-PhilsLab:BGA96C80P9X16_900X1300X120"
+		(property "Footprint" "easyeda2kicad_foorprint:FBGA-96_L14.0-W8.0-R16-C6-P0.80-TL"
 			(at 189.23 100.33 0)
 			(effects
@@
 			)
 		)
+		(property "LCSC" "C367428"
+			(at 189.23 100.33 0)
+			(effects
+				(font
+					(size 1.27 1.27)
+				)
+				(hide yes)
+			)
+		)
+		(property "Manufacturer Part Number" "MT41K256M16TW-107 IT:P"
+			(at 189.23 100.33 0)
+			(effects
+				(font
+					(size 1.27 1.27)
+				)
+				(hide yes)
+			)
+		)
 		(pin "J9"
 		)
@@
 			)
 		)
-		(property "Footprint" "Footprint-Lib-PhilsLab:BGA96C80P9X16_900X1300X120"
+		(property "Footprint" "easyeda2kicad_foorprint:FBGA-96_L14.0-W8.0-R16-C6-P0.80-TL"
 			(at 203.2 195.58 0)
 			(effects
@@
 			)
 		)
+		(property "LCSC" "C367428"
+			(at 203.2 195.58 0)
+			(effects
+				(font
+					(size 1.27 1.27)
+				)
+				(hide yes)
+			)
+		)
+		(property "Manufacturer Part Number" "MT41K256M16TW-107 IT:P"
+			(at 203.2 195.58 0)
+			(effects
+				(font
+					(size 1.27 1.27)
+				)
+				(hide yes)
+			)
+		)
 		(pin "J9"
 		)
@@
 			)
 		)
-		(property "Footprint" "Footprint-Lib-PhilsLab:BGA96C80P9X16_900X1300X120"
+		(property "Footprint" "easyeda2kicad_foorprint:FBGA-96_L14.0-W8.0-R16-C6-P0.80-TL"
 			(at 50.8 25.4 0)
 			(effects
@@
 			)
 		)
+		(property "LCSC" "C367428"
+			(at 50.8 25.4 0)
+			(effects
+				(font
+					(size 1.27 1.27)
+				)
+				(hide yes)
+			)
+		)
+		(property "Manufacturer Part Number" "MT41K256M16TW-107 IT:P"
+			(at 50.8 25.4 0)
+			(effects
+				(font
+					(size 1.27 1.27)
+				)
+				(hide yes)
+			)
+		)
 		(pin "J9"
 		)
@@
 			)
 		)
-		(property "Footprint" "Footprint-Lib-PhilsLab:BGA96C80P9X16_900X1300X120"
+		(property "Footprint" "easyeda2kicad_foorprint:FBGA-96_L14.0-W8.0-R16-C6-P0.80-TL"
 			(at 199.39 125.73 0)
 			(effects
@@
 			)
 		)
+		(property "LCSC" "C367428"
+			(at 199.39 125.73 0)
+			(effects
+				(font
+					(size 1.27 1.27)
+				)
+				(hide yes)
+			)
+		)
+		(property "Manufacturer Part Number" "MT41K256M16TW-107 IT:P"
+			(at 199.39 125.73 0)
+			(effects
+				(font
+					(size 1.27 1.27)
+				)
+				(hide yes)
+			)
+		)
 		(pin "J9"
 		)
@@
 			)
 		)
-		(property "Footprint" "Footprint-Lib-PhilsLab:BGA96C80P9X16_900X1300X120"
+		(property "Footprint" "easyeda2kicad_foorprint:FBGA-96_L14.0-W8.0-R16-C6-P0.80-TL"
 			(at 54.61 114.3 0)
 			(effects
@@
 				(hide yes)
 			)
+		)
+		(property "LCSC" "C367428"
+			(at 54.61 114.3 0)
+			(effects
+				(font
+					(size 1.27 1.27)
+				)
+				(hide yes)
+			)
+		)
+		(property "Manufacturer Part Number" "MT41K256M16TW-107 IT:P"
+			(at 54.61 114.3 0)
+			(effects
+				(font
+					(size 1.27 1.27)
+				)
+				(hide yes)
+			)
