File: zynq_soc_board_v1.kicad_pcb (KiCad board)
At the start: 10 copper layers, 418 parts, among them J100 CON-SOCJ-2155, J1000 10144518-082802LF, J1001 10144518-082802LF, J300 Digilent HS2 Header, J301 USB-MICRO-B, J800 HR911130A, J900 U-M-M5DW-W-1, Q100 T2N7002AK, Q300 T2N7002AK, Q400 T2N7002AK, Q500 T2N7002AK, SW300 SKRPANE010, SW301 219-3LPST, SW400 SKRPANE010, U100 LS1205EVD33, U101 SY8003ADFC, U102 SY8003ADFC, U103 SY8003ADFC, U104 SY8003ADFC, U105 BD3539FVM-TR, U300 FT2232HL-REEL, U301 93LC56BT-I/SN, U400 SN74LVC1G07DRLR, U401 SN74LVC1G07DRLR, U402 W25Q128JVEIQ, U403 MTFC8GAKAJCN-4M_IT, U6 XC7Z020-2CLG400I, U700 MT41K256M16TW-107 IT:P, U701 MT41K256M16TW-107 IT:P, U800 RTL8211F-CG, U900 USB3320C-EZK-TR, X300 12Mhz-TXC Corp, X400 ECS-2520MV-33.3, X800 ECS-2520MV-250, X900 ECS-2520MV-130-BN

Commit message: xc7z020-fanout
Parts:
- added H1: MountingHole, MountingHole:MountingHole_3.2mm_M3, F.Cu at (200.9, 61.9)
- added H2: MountingHole, MountingHole:MountingHole_3.2mm_M3, F.Cu at (113.5, 61.4)
- added H3: MountingHole, MountingHole:MountingHole_3.2mm_M3, F.Cu at (113.7, 118.3)
- added H4: MountingHole, MountingHole:MountingHole_3.2mm_M3, F.Cu at (200.8, 118.2)
- J1000, J1001, J301, SW301: moved to B.Cu
- U6: footprint zynq_sc7z0x0:CLG400 -> Package_BGA:Xilinx_CLG400
- moved FB300 261.8 mm to (256.0, 80.7)
- moved FB301 261.8 mm to (256.0, 83.2)
- moved FB302 261.8 mm to (256.0, 85.8)
- moved Q300 248.5 mm to (264.9, 111.2)
- moved C233 235.9 mm to (282.9, 68.2)
- moved C234 235.9 mm to (282.9, 71.6)
- moved C235 235.9 mm to (282.9, 75.0)
- moved C248 235.9 mm to (282.9, 78.3)
- moved C300 235.9 mm to (250.2, 94.5)
- moved C301 235.9 mm to (250.2, 96.5)
- moved C302 235.9 mm to (250.2, 98.4)
- moved C303 235.9 mm to (250.2, 100.4)
- moved C304 235.9 mm to (250.2, 102.4)
- moved C305 235.9 mm to (250.2, 104.3)
- moved C306 235.9 mm to (250.2, 106.3)
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Routing:
- net GND: track 0.00 -> 49.4 mm, vias 0 -> 55
- net +3V3: track 0.00 -> 16.4 mm, vias 0 -> 20
- net +1V0: track 0.00 -> 13.2 mm, vias 0 -> 9
- net +1V8: track 0.00 -> 12.7 mm, vias 0 -> 13
- net /zynq_jtag/NINIT: track 0.00 -> 7.51 mm
- net +1V35: track 0.00 -> 6.76 mm, vias 0 -> 10
- net DONE: track 0.00 -> 6.35 mm
- net /zynq_programmable_logic/NPUDC: track 0.00 -> 4.66 mm
- net /zynq_ddr/DDR_DQ0: track 0.00 -> 4.11 mm
- net /zynq_processing_system_ps/ETH_NRST: track 0.00 -> 3.59 mm
- net QSPI_DQ0_M3: track 0.00 -> 3.38 mm
- net MIO51: track 0.00 -> 3.35 mm
- net QSPI_DQ2_M2: track 0.00 -> 3.34 mm
- net PS_NRST: track 0.00 -> 3.33 mm
- net UART1_RX: track 0.00 -> 3.32 mm
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Other:
- board outline added: 95.1 x 64.6 mm

Commit message: ram-update
Parts:
- added C226: 470n, easyeda2kicad_foorprint:C0201, F.Cu at (85.9, 124.3)
- added C227: 470n, easyeda2kicad_foorprint:C0201, F.Cu at (85.9, 126.0)
- added C238: 470n, easyeda2kicad_foorprint:C0201, F.Cu at (88.4, 122.5)
- added C240: 470n, easyeda2kicad_foorprint:C0201, F.Cu at (88.4, 126.0)
- added C241: 470n, easyeda2kicad_foorprint:C0201, F.Cu at (90.8, 119.0)
- added C242: 470n, easyeda2kicad_foorprint:C0201, F.Cu at (90.8, 120.8)
- added C245: 470n, easyeda2kicad_foorprint:C0201, F.Cu at (90.8, 126.0)
- added C707: 47n, easyeda2kicad_foorprint:C0201, F.Cu at (96.7, 88.8)
- added C711: 47n, easyeda2kicad_foorprint:C0201, F.Cu at (99.0, 85.0)
- added C715: 47n, easyeda2kicad_foorprint:C0201, F.Cu at (99.0, 88.8)
- added C720: 47n, easyeda2kicad_foorprint:C0201, F.Cu at (100.1, 81.8)
- added C722: 47n, easyeda2kicad_foorprint:C0201, B.Cu at (126.0, 103.5)
- added C723: 47n, easyeda2kicad_foorprint:C0201, B.Cu at (130.1, 97.0)
- C201, C205, C210, C216, C220, C223, C229, C232, C235, C236, C400, C608, C609, C610, C611, R427: moved to B.Cu
- C202, C203, C206, C207, C208, C214, C215, C217, C218, C219, C222, C225, C228, C231, C239, C243, C600, C601, C602, C603, C604, C605, C606, C607, C612, C613, C700, C701, C703, C704, C705, C706, C707, C708, C709, C710, C711, C713, C714, C715, C716, C717, C718, C719, C720, C721: footprint Capacitor_SMD:C_0402_1005Metric -> easyeda2kicad_foorprint:C0201; moved to B.Cu
- C211, C226, C227, C238, C240, C241, C242, C244, C245, C712: footprint Capacitor_SMD:C_0402_1005Metric -> easyeda2kicad_foorprint:C0201
- C725, C726, C727, C728, C729, C730, C731, C732, C733, C735, C736, C737, C738, C739, C740, C741, C742, C743: footprint Capacitor_SMD:C_0402_1005Metric -> Capacitor_SMD:C_0201_0603Metric; moved to B.Cu
- R310, R312, R314, R316, R319, R404, R405: footprint Resistor_SMD:R_0402_1005Metric -> easyeda2kicad_foorprint:R0201
- R600, R601, R602, R603, R604, R605, R606, R607, R608, R609, R610, R611, R612, R613, R614, R615, R616, R617, R618, R619, R620, R621, R622, R623, R624, R626, R627: footprint Resistor_SMD:R_0402_1005Metric -> easyeda2kicad_foorprint:R0201; moved to B.Cu
- moved C244 149.2 mm to (90.8, 124.3)
- moved C211 136.1 mm to (83.2, 115.5)
- moved Q400 126.1 mm to (134.7, 76.1), turned to 90 degrees
- moved C235 108.8 mm to (174.8, 62.6), turned to -90 degrees
- moved R427 99.0 mm to (151.2, 86.7), turned to -90 degrees
- moved C400 95.9 mm to (151.2, 89.9), turned to 90 degrees
- moved C231 85.4 mm to (148.1, 93.5), turned to 45 degrees
- moved C232 84.9 mm to (149.2, 95.9)
- moved C225 84.1 mm to (143.5, 95.6), turned to 135 degrees
- moved C243 83.5 mm to (155.7, 97.4)
- moved C222 83.4 mm to (150.0, 97.4), turned to 180 degrees
- moved C223 82.6 mm to (150.1, 98.2), turned to 180 degrees
- moved C229 81.8 mm to (142.0, 97.8), turned to 180 degrees
- moved C220 81.0 mm to (152.0, 93.9), turned to 90 degrees
- moved C613 77.8 mm to (148.0, 95.1), turned to 45 degrees
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- renumbered C1 to C105
Routing:
- net GND: track 49.4 -> 88.4 mm, vias 55 -> 98
- net +1V35: track 6.76 -> 37.8 mm, vias 10 -> 46
- net /zynq_ddr/DDR_A10: track 0.56 -> 9.78 mm, vias 1 -> 2
- net /zynq_ddr/DDR_A12: track 0.58 -> 6.89 mm
- net /zynq_ddr/DDR_A1: track 2.17 -> 8.04 mm
- net /zynq_ddr/DDR_BA0: track 0.55 -> 5.53 mm
- net /zynq_ddr/DDR_A2: track 0.58 -> 5.18 mm, vias 1 -> 3
- net /zynq_ddr/DDR_DQ5: track 1.36 -> 5.93 mm
- net /zynq_ddr/DDR_NRST: track 3.28 -> 7.67 mm, vias 0 -> 2
- net /zynq_ddr/DDR_A5: track 0.99 -> 5.13 mm, vias 0 -> 2
- net /zynq_ddr/DDR_BA2: track 0.56 -> 4.34 mm
- net /zynq_ddr/DDR_ZQ2: track 0.00 -> 3.20 mm
- net /zynq_ddr/DDR_ZQ1: track 0.00 -> 3.18 mm
- net /zynq_ddr/DDR_A9: track 0.56 -> 3.66 mm
- net /zynq_ddr/DDR_NWE: track 0.57 -> 3.51 mm, vias 1 -> 3
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
Commit message: ram-zynq-updated
Parts:
- removed the C226 at (207.2, 42.6)
- removed the C227 at (207.2, 44.6)
- removed the C238 at (210.1, 42.6)
- removed the C240 at (210.1, 46.5)
- removed the C241 at (210.1, 48.5)
- removed the C242 at (218.0, 29.8)
- removed the C245 at (212.9, 40.6)
- removed the C707 at (96.7, 88.8)
- removed the C711 at (99.0, 85.0)
- removed the C715 at (99.0, 88.8)
- removed the C720 at (100.1, 81.8)
- C100, C101, C102, C103, C130, C200, C204, C211, C213, C221, C224, C226, C227, C233, C237, C238, C240, C241, C242, C244, C245, C246, C247, C301, C302, C316, C402, C403, C405, C406, C407, C408, C409, C410, C800, C801, C802, C803, C804, C805, C806, C812, C813, C814, C815, C816, C817, C818, C819, C901, C902, C903, C904, D306, D900, D901, FB200, FB300, FB800, FB801, R100, R101, R102, R128, R324, R325, R326, R327, R328, R333, R334, R335, R400, R401, R403, R404, R405, R420, R903, U100, U301, U400, X400: moved to B.Cu
- D305: footprint Diode_SMD:D_SOD-323F -> easyeda2kicad_foorprint:SOD-323_L1.8-W1.3-LS2.5-RD; moved to B.Cu
- moved C233 148.8 mm to (140.2, 110.3), turned to 180 degrees
- moved C204 142.8 mm to (140.1, 107.9), turned to 180 degrees
- moved C209 139.6 mm to (138.1, 61.7), turned to 90 degrees
- moved R128 135.3 mm to (197.2, 73.0), turned to 180 degrees
- moved C102 135.3 mm to (181.1, 110.6), turned to -90 degrees
- moved C101 135.1 mm to (180.2, 110.6), turned to -90 degrees
- moved D400 134.1 mm to (134.8, 67.5)
- moved R101 131.0 mm to (183.2, 110.6), turned to -90 degrees
- moved R102 129.6 mm to (182.2, 110.7), turned to 90 degrees
- moved R100 129.2 mm to (180.6, 112.2), turned to 180 degrees
- moved R412 121.3 mm to (134.8, 65.4)
- moved C100 119.3 mm to (184.7, 107.3), turned to 90 degrees
- moved R414 119.3 mm to (135.7, 71.4), turned to 180 degrees
- moved U401 119.1 mm to (138.5, 74.0)
- moved R413 118.8 mm to (135.7, 70.3)
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Connections:
- net /ethernet_gigabit/ETH_PHY_RXCLK renamed ETH_PHY_RXCLK
- net /ethernet_gigabit/ETH_PHY_RXCTL renamed ETH_PHY_RXCTL
- net /ethernet_gigabit/ETH_PHY_RXD0 renamed ETH_PHY_RXD0
- net /ethernet_gigabit/ETH_PHY_RXD1 renamed ETH_PHY_RXD1
- net /ethernet_gigabit/ETH_PHY_RXD2 renamed ETH_PHY_RXD2
- net /ethernet_gigabit/ETH_PHY_RXD3 renamed ETH_PHY_RXD3
- net /ethernet_gigabit/MDI0_N renamed MDI0_N
- net /ethernet_gigabit/MDI0_P renamed MDI0_P
- net /ethernet_gigabit/MDI1_N renamed MDI1_N
- net /ethernet_gigabit/MDI1_P renamed MDI1_P
- net /ethernet_gigabit/MDI2_N renamed MDI2_N
- net /ethernet_gigabit/MDI2_P renamed MDI2_P
- net /ethernet_gigabit/MDI3_N renamed MDI4_N
- net /ethernet_gigabit/MDI3_P renamed MDI3_P
- net /zynq_ddr/DDR_A0 renamed DDR_A0
- net /zynq_ddr/DDR_A1 renamed DDR_A1
- net /zynq_ddr/DDR_A10 renamed DDR_A10
- net /zynq_ddr/DDR_A11 renamed DDR_A11
- net /zynq_ddr/DDR_A12 renamed DDR_A12
- net /zynq_ddr/DDR_A13 renamed DDR_A13
- net /zynq_ddr/DDR_A14 renamed DDR_A14
- net /zynq_ddr/DDR_A2 renamed DDR_A2
- net /zynq_ddr/DDR_A3 renamed DDR_A3
- net /zynq_ddr/DDR_A4 renamed DDR_A4
- net /zynq_ddr/DDR_A5 renamed DDR_A5
- net /zynq_ddr/DDR_A6 renamed DDR_A6
- net /zynq_ddr/DDR_A7 renamed DDR_A7
- net /zynq_ddr/DDR_A8 renamed DDR_A8
- net /zynq_ddr/DDR_A9 renamed DDR_A9
- net /zynq_ddr/DDR_BA0 renamed DDR_BA0
- net /zynq_ddr/DDR_BA1 renamed DDR_BA1
- net /zynq_ddr/DDR_BA2 renamed DDR_BA2
- net /zynq_ddr/DDR_CKE renamed DDR_CKE
- net /zynq_ddr/DDR_CK_N renamed DDR_CK_N
- net /zynq_ddr/DDR_CK_P renamed DDR_CK_P
- net /zynq_ddr/DDR_DM0 renamed DDR_DM0
- net /zynq_ddr/DDR_DM1 renamed DDR_DM1
- net /zynq_ddr/DDR_DM2 renamed DDR_DM2
- net /zynq_ddr/DDR_DM3 renamed DDR_DM3
- net /zynq_ddr/DDR_DQ0 renamed DDR_DQ0
- net /zynq_ddr/DDR_DQ1 renamed DDR_DQ1
- net /zynq_ddr/DDR_DQ10 renamed DDR_DQ10
- net /zynq_ddr/DDR_DQ11 renamed DDR_DQ11
- net /zynq_ddr/DDR_DQ12 renamed DDR_DQ12
- net /zynq_ddr/DDR_DQ13 renamed DDR_DQ13
- net /zynq_ddr/DDR_DQ14 renamed DDR_DQ14
- net /zynq_ddr/DDR_DQ15 renamed DDR_DQ15
- net /zynq_ddr/DDR_DQ16 renamed DDR_DQ16
- net /zynq_ddr/DDR_DQ17 renamed DDR_DQ17
- net /zynq_ddr/DDR_DQ18 renamed DDR_DQ18
- net /zynq_ddr/DDR_DQ19 renamed DDR_DQ19
- net /zynq_ddr/DDR_DQ2 renamed DDR_DQ2
- net /zynq_ddr/DDR_DQ20 renamed DDR_DQ20
- net /zynq_ddr/DDR_DQ21 renamed DDR_DQ21
- net /zynq_ddr/DDR_DQ22 renamed DDR_DQ22
- net /zynq_ddr/DDR_DQ23 renamed DDR_DQ23
- net /zynq_ddr/DDR_DQ24 renamed DDR_DQ24
- net /zynq_ddr/DDR_DQ25 renamed DDR_DQ25
- net /zynq_ddr/DDR_DQ26 renamed DDR_DQ26
- net /zynq_ddr/DDR_DQ27 renamed DDR_DQ27
- net /zynq_ddr/DDR_DQ28 renamed DDR_DQ28
- net /zynq_ddr/DDR_DQ29 renamed DDR_DQ29
- net /zynq_ddr/DDR_DQ3 renamed DDR_DQ3
- net /zynq_ddr/DDR_DQ30 renamed DDR_DQ30
- net /zynq_ddr/DDR_DQ31 renamed DDR_DQ31
- net /zynq_ddr/DDR_DQ4 renamed DDR_DQ4
- net /zynq_ddr/DDR_DQ5 renamed DDR_DQ5
- net /zynq_ddr/DDR_DQ6 renamed DDR_DQ6
- net /zynq_ddr/DDR_DQ7 renamed DDR_DQ7
- net /zynq_ddr/DDR_DQ8 renamed DDR_DQ8
- net /zynq_ddr/DDR_DQ9 renamed DDR_DQ9
- net /zynq_ddr/DDR_DQS0_N renamed DDR_DQS0_N
- net /zynq_ddr/DDR_DQS0_P renamed DDR_DQS0_P
- net /zynq_ddr/DDR_DQS1_N renamed DDR_DQS1_N
- net /zynq_ddr/DDR_DQS1_P renamed DDR_DQS1_P
- net /zynq_ddr/DDR_DQS2_N renamed DDR_DQS2_N
- net /zynq_ddr/DDR_DQS2_P renamed DDR_DQS2_P
- net /zynq_ddr/DDR_DQS3_N renamed DDR_DQS3_N
- net /zynq_ddr/DDR_DQS3_P renamed DDR_DQS3_P
- net /zynq_ddr/DDR_NCAS renamed DDR_NCAS
- net /zynq_ddr/DDR_NCS renamed DDR_NCS
- net /zynq_ddr/DDR_NRAS renamed DDR_NRAS
- net /zynq_ddr/DDR_NRST renamed DDR_NRST
- net /zynq_ddr/DDR_NWE renamed DDR_NWE
- net /zynq_ddr/DDR_ODT renamed DDR_ODT
Routing:
- net DDR_CK_N: track 1.74 -> 83.8 mm
- net DDR_CK_P: track 2.33 -> 82.5 mm
- net DDR_A5: track 5.13 -> 64.8 mm, vias 2 -> 3
- net DDR_A7: track 1.73 -> 61.3 mm
- net DDR_A3: track 4.11 -> 62.9 mm, vias 2 -> 3
- net DDR_BA0: track 5.53 -> 61.3 mm, vias 1 -> 2
- net DDR_A9: track 3.66 -> 58.6 mm, vias 1 -> 2
- net DDR_BA2: track 4.34 -> 58.1 mm, vias 1 -> 2
- net DDR_NCAS: track 1.72 -> 55.0 mm
- net DDR_A0: track 4.59 -> 57.8 mm, vias 2 -> 3
- net DDR_A8: track 2.63 -> 55.4 mm, vias 1 -> 3
- net DDR_CKE: track 5.34 -> 58.0 mm, vias 1 -> 3
- net DDR_NCS: track 2.48 -> 54.4 mm, vias 2 -> 3
- net DDR_NRAS: track 1.73 -> 53.5 mm
- net DDR_A4: track 1.72 -> 52.0 mm
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
Commit message: ram_ended
Parts:
- moved R701 0.52 mm to (126.0, 105.9)
- moved C705 0.31 mm to (126.6, 82.1)
- moved C740 0.16 mm to (133.6, 105.8)
Routing:
- net DDR_A14: track 1.86 -> 89.2 mm, vias 2 -> 3
- net DDR_A11: track 3.50 -> 89.3 mm, vias 2 -> 3
- net DDR_ODT: track 4.26 -> 89.1 mm
- net DDR_A12: track 6.89 -> 89.1 mm, vias 1 -> 3
- net DDR_A10: track 9.78 -> 89.1 mm, vias 2 -> 3
- net DDR_A13: track 10.6 -> 89.1 mm, vias 2 -> 3
- net DDR_BA1: track 50.5 -> 88.9 mm
- net DDR_A6: track 50.6 -> 88.9 mm
- net DDR_A4: track 52.0 -> 89.0 mm
- net DDR_NWE: track 52.8 -> 89.1 mm
- net DDR_NRAS: track 53.5 -> 89.0 mm
- net DDR_A2: track 54.2 -> 89.2 mm
- net DDR_NCS: track 54.4 -> 89.3 mm
- net DDR_NCAS: track 55.0 -> 88.9 mm
- net DDR_A8: track 55.4 -> 89.1 mm
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