File: zynq_soc_board_v1.kicad_pcb (KiCad board)
At the start: 10 copper layers, 95.1 x 64.6 mm, 424 parts, among them J100 CON-SOCJ-2155, J1000 10144518-082802LF, J1001 10144518-082802LF, J300 Digilent HS2 Header, J301 USB-MICRO-B, J800 HR911130A, J900 U-M-M5DW-W-1, Q100 T2N7002AK, Q300 T2N7002AK, Q400 T2N7002AK, Q500 T2N7002AK, SW300 SKRPANE010, SW301 219-3LPST, SW400 SKRPANE010, U100 LS1205EVD33, U101 SY8003ADFC, U102 SY8003ADFC, U103 SY8003ADFC, U104 SY8003ADFC, U105 BD3539FVM-TR, U300 FT2232HL-REEL, U301 93LC56BT-I/SN, U400 SN74LVC1G07DRLR, U401 SN74LVC1G07DRLR, U402 W25Q128JVEIQ, U403 MTFC8GAKAJCN-4M_IT, U6 XC7Z020-2CLG400I, U700 MT41K256M16TW-107 IT:P, U701 MT41K256M16TW-107 IT:P, U800 RTL8211F-CG, U900 USB3320C-EZK-TR, X300 12Mhz-TXC Corp, X400 ECS-2520MV-33.3, X800 ECS-2520MV-250, X900 ECS-2520MV-130-BN

Commit message: pcb_eth
Parts:
- C100, C103, C104, C107, C108, C109, C112, C113, C114, C117, C118, C119, C122, C123, C124, C127: footprint Footprint-Lib-PhilsLab:CAP_0805 -> easyeda2kicad_foorprint:C0805
- C734: moved to B.Cu
- L100, L101, L102, L103: footprint Footprint-Lib-PhilsLab:SRP0415 -> easyeda2kicad_foorprint:IND-SMD_L4.4-W4.1
- U101, U102, U103, U104: footprint Footprint-Lib-PhilsLab:DFN2x2-8 -> easyeda2kicad_foorprint:DFN-8_L2.0-W2.0-P0.50-LS2.0-BL-EP
- U403: footprint MTFC8GAKAJCN-4M_IT:BGA153N50P14X14_1150X1300X100 -> easyeda2kicad_foorprint:FBGA-153_L13.0-W11.5-P0.50_KLMAG1JETD-B041
- U700, U701: footprint Footprint-Lib-PhilsLab:BGA96C80P9X16_900X1300X120 -> easyeda2kicad_foorprint:FBGA-96_L14.0-W8.0-R16-C6-P0.80-TL
- U800: footprint Footprint-Lib-PhilsLab:QFN-40-0.4-EP -> easyeda2kicad_foorprint:WQFN-40_L5.0-W5.0-P0.4-BL-EP
- moved R115 146.7 mm to (127.5, 117.4), turned to 90 degrees
- moved C120 138.7 mm to (185.8, 117.4)
- moved C121 136.0 mm to (182.8, 119.5)
- moved R118 129.3 mm to (185.8, 119.5)
- moved R119 128.6 mm to (185.8, 118.4), turned to 180 degrees
- moved R107 126.5 mm to (146.4, 117.4)
- moved R121 124.8 mm to (182.8, 118.4), turned to 180 degrees
- moved R122 124.3 mm to (182.8, 117.4)
- moved C110 123.4 mm to (167.1, 117.3)
- moved C111 122.9 mm to (164.3, 119.5)
- moved R120 122.3 mm to (180.0, 117.4), turned to 90 degrees
- moved R108 115.3 mm to (167.1, 119.5)
- moved R109 114.4 mm to (167.1, 118.4), turned to 180 degrees
- moved L800 112.4 mm to (173.6, 82.7), turned to 90 degrees
- moved C105 111.6 mm to (149.6, 117.3)
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Connections:
- C107 pad 2: Net-(C107-Pad2) -> GND
- C108 pad 2: Net-(C107-Pad2) -> GND
- C112 pad 2: Net-(C112-Pad2) -> GND
- C113 pad 2: Net-(C112-Pad2) -> GND
- C117 pad 2: Net-(C117-Pad2) -> GND
- C118 pad 2: Net-(C117-Pad2) -> GND
- C122 pad 2: Net-(C122-Pad2) -> GND
- C123 pad 2: Net-(C122-Pad2) -> GND
Routing:
- net GND: track 94.2 -> 127.3 mm, vias 102 -> 148
- net DDR_DQ13: track 1.10 -> 24.6 mm
- net DDR_DQ10: track 1.12 -> 24.6 mm
- net DDR_DQ11: track 1.13 -> 24.6 mm
- net DDR_DQ9: track 2.48 -> 24.7 mm
- net DDR_DQS1_N: track 3.50 -> 24.7 mm
- net DDR_DM1: track 3.60 -> 24.6 mm
- net DDR_DQS1_P: track 4.24 -> 24.8 mm
- net DDR_DQ8: track 4.22 -> 24.7 mm
- net DDR_DQ18: track 1.09 -> 21.4 mm
- net DDR_DQS2_N: track 1.17 -> 21.5 mm
- net DDR_DQS2_P: track 1.18 -> 21.4 mm
- net DDR_DQ20: track 1.15 -> 21.3 mm
- net DDR_DQ16: track 1.72 -> 21.4 mm, vias 1 -> 2
- net DDR_DQ19: track 1.72 -> 21.3 mm, vias 1 -> 2
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- added copper zone on F.Cu, net +0V675
- added copper zone on F.Cu, net +1V0
- added copper zone on F.Cu, net +1V35
- added copper zone on F.Cu, net +1V8
- added copper zone on F.Cu, net +3V3
- added copper zone on F.Cu, net +5V
- added copper zone on F.Cu, net /power/SW_1V0
- added copper zone on F.Cu, net /power/SW_1V35
- added copper zone on F.Cu, net /power/SW_1V8
- added copper zone on F.Cu, net /power/SW_3V3
- added copper zone on F.Cu, net GND
