File: USB-2-HS.kicad_sch (KiCad schematic)
At the start: 24 parts, among them J900 U-M-M5DW-W-1, U900 USB3320C-EZK-TR, U901 MIC2099-1YMT-TR, X900 ECS-2520MV-130-BN

Commit message: rev a done
Parts:
- X900: footprint Footprint-Lib-PhilsLab:XTAL_2520 -> Crystal:Crystal_SMD_2520-4Pin_2.5x2.0mm
Changed lines of the file:
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@@
 			)
 		)
-		(property "Footprint" "Footprint-Lib-PhilsLab:XTAL_2520"
+		(property "Footprint" "Crystal:Crystal_SMD_2520-4Pin_2.5x2.0mm"
 			(at 43.18 104.14 0)
 			(effects
