File: ethernet.kicad_sch (KiCad schematic)
At the start: 50 parts, among them J800 HR911130A, U800 RTL8211F-CG, X800 ECS-2520MV-250

Commit message: pcbb
Connections:
- net CGND: now reaches J800.SH (SHIELD)
- no-connect marks 2 -> 1
Changed lines of the file:
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@@
 		(at 271.78 83.82)
 	)
-	(no_connect
-		(at 256.54 102.87)
-	)
 	(wire
 		(pts
@@
 					(unit 1)
 				)
+			)
+		)
+	)
+	(symbol
+		(lib_id "power:Earth")
+		(at 256.54 102.87 0)
+		(unit 1)
+		(exclude_from_sim no)
+		(in_bom yes)
+		(on_board yes)
+		(dnp no)
+		(property "Reference" "#PWR073"
+			(at 256.54 109.22 0)
+			(effects
+				(font
+					(size 1.27 1.27)
+				)
+				(hide yes)
+			)
+		)
+		(property "Value" "CGND"
+			(at 256.54 106.934 0)
+			(effects
+				(font
+					(size 1.27 1.27)
+				)
+			)
+		)
+		(property "Footprint" ""
+			(at 256.54 102.87 0)
+			(effects
+				(font
+					(size 1.27 1.27)
+				)
+				(hide yes)
+			)
+		)
+		(property "Datasheet" "~"
+			(at 256.54 102.87 0)
+			(effects
+				(font
+					(size 1.27 1.27)
+				)
+				(hide yes)
+			)
+		)
+		(property "Description" "Power symbol creates a global label with name \"Earth\""
+			(at 256.54 102.87 0)
+			(effects
+				(font
+					(size 1.27 1.27)
+				)
+				(hide yes)
+			)
+		)
+		(pin "1"
+		)
+		(instances
+			(project "zynq_soc_board_v1"
+				(path "/068a81e1-1783-4521-9958-788ddeed3b49/ae319a65-0a6c-4d0b-b442-f6b6cf9cba1c"
+					(reference "#PWR073")
+					(unit 1)
+				)

Commit message: rev a done
Parts:
- X800: footprint Footprint-Lib-PhilsLab:XTAL_2520 -> Crystal:Crystal_SMD_2520-4Pin_2.5x2.0mm
Changed lines of the file:
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@@
 			)
 		)
-		(property "Footprint" "Footprint-Lib-PhilsLab:XTAL_2520"
+		(property "Footprint" "Crystal:Crystal_SMD_2520-4Pin_2.5x2.0mm"
 			(at 38.1 124.46 0)
 			(effects
