File: Mezzanine Connectors.kicad_sch (KiCad schematic)
At the start: 2 parts, among them J1000 10144518-082802LF, J1001 10144518-082802LF

Commit message: all page
Connections:
- net PL_B34_L4_N: no longer J1001.65
- new net PL_B34_L4_P: J1001.65
- no-connect marks 4 -> 10
Other:
- title: (none) -> Mezzanine Connectors

Commit message: sch-to-pcb
Connections:
- net PL_B35_L11_P renamed PL_B35_L11_N

Commit message: pcb layers
Connections:
- net MIO44: now reaches J1000.69
- net MIO46: now reaches J1000.70
- net MIO45: now reaches J1000.71
- net MIO47: now reaches J1000.72
- net MIO43: now reaches J1000.77
- net MIO48: now reaches J1000.78
- no-connect marks 10 -> 4
Changed lines of the file:
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@@
 	)
 	(no_connect
-		(at 59.69 135.89)
-	)
-	(no_connect
-		(at 74.93 135.89)
-	)
-	(no_connect
 		(at 59.69 67.31)
 	)
 	(no_connect
-		(at 59.69 128.27)
-	)
-	(no_connect
 		(at 59.69 87.63)
 	)
 	(no_connect
-		(at 59.69 125.73)
-	)
-	(no_connect
-		(at 74.93 128.27)
-	)
-	(no_connect
 		(at 59.69 64.77)
 	)
-	(no_connect
-		(at 74.93 125.73)
-	)
 	(wire
 		(pts
@@
 	(wire
 		(pts
+			(xy 41.91 135.89) (xy 59.69 135.89)
+		)
+		(stroke
+			(width 0)
+			(type default)
+		)
+	)
+	(wire
+		(pts
 			(xy 160.02 81.28) (xy 175.26 81.28)
 		)
@@
 	(wire
 		(pts
+			(xy 83.82 125.73) (xy 74.93 125.73)
+		)
+		(stroke
+			(width 0)
+			(type default)
+		)
+	)
+	(wire
+		(pts
 			(xy 190.5 127) (xy 203.2 127)
 		)
@@
 	(wire
 		(pts
+			(xy 83.82 128.27) (xy 74.93 128.27)
+		)
+		(stroke
+			(width 0)
+			(type default)
+		)
+	)
+	(wire
+		(pts
 			(xy 171.45 132.08) (xy 171.45 124.46)
 		)
@@
 	(wire
 		(pts
+			(xy 41.91 128.27) (xy 59.69 128.27)
+		)
+		(stroke
+			(width 0)
+			(type default)
+		)
+	)
+	(wire
+		(pts
 			(xy 203.2 137.16) (xy 190.5 137.16)
 		)
@@
 	(wire
 		(pts
+			(xy 83.82 135.89) (xy 74.93 135.89)
+		)
+		(stroke
+			(width 0)
+			(type default)
+		)
+	)
+	(wire
+		(pts
 			(xy 194.31 55.88) (xy 194.31 63.5)
 		)
@@
 	(wire
 		(pts
+			(xy 41.91 125.73) (xy 59.69 125.73)
+		)
+		(stroke
+			(width 0)
+			(type default)
+		)
+	)
+	(wire
+		(pts
 			(xy 74.93 120.65) (xy 82.55 120.65)
 		)
@@
 		)
 	)
+	(global_label "MIO44"
+		(shape input)
+		(at 41.91 125.73 180)
+		(fields_autoplaced yes)
+		(effects
+			(font
+				(size 0.762 0.762)
+				(thickness 0.254)
+				(bold yes)
+			)
+			(justify right)
+		)
+		(property "Intersheetrefs" "${INTERSHEET_REFS}"
+			(at 36.1591 125.73 0)
+			(effects
+				(font
+					(size 1.27 1.27)
+				)
+				(justify right)
+				(hide yes)
+			)
+		)
+	)
 	(global_label "PL_B35_L6_P"
 		(shape input)
@@
 		)
 	)
+	(global_label "MIO46"
+		(shape input)
+		(at 83.82 125.73 0)
+		(fields_autoplaced yes)
+		(effects
+			(font
+				(size 0.762 0.762)
+				(thickness 0.254)
+				(bold yes)
+			)
+			(justify left)
+		)
+		(property "Intersheetrefs" "${INTERSHEET_REFS}"
+			(at 89.5709 125.73 0)
+			(effects
+				(font
+					(size 1.27 1.27)
+				)
+				(justify left)
+				(hide yes)
+			)
+		)
+	)
 	(global_label "PL_B35_IO25"
 		(shape input)
@@
 		)
 	)
+	(global_label "MIO47"
+		(shape input)
+		(at 83.82 128.27 0)
+		(fields_autoplaced yes)
+		(effects
+			(font
+				(size 0.762 0.762)
+				(thickness 0.254)
+				(bold yes)
+			)
+			(justify left)
+		)
+		(property "Intersheetrefs" "${INTERSHEET_REFS}"
+			(at 89.5709 128.27 0)
+			(effects
+				(font
+					(size 1.27 1.27)
+				)
+				(justify left)
+				(hide yes)
+			)
+		)
+	)
 	(global_label "PL_B35_L6_N"
 		(shape input)
@@
 		)
 	)
+	(global_label "MIO48"
+		(shape input)
+		(at 83.82 135.89 0)
+		(fields_autoplaced yes)
+		(effects
+			(font
+				(size 0.762 0.762)
+				(thickness 0.254)
+				(bold yes)
+			)
+			(justify left)
+		)
+		(property "Intersheetrefs" "${INTERSHEET_REFS}"
+			(at 89.5709 135.89 0)
+			(effects
+				(font
+					(size 1.27 1.27)
+				)
+				(justify left)
+				(hide yes)
+			)
+		)
+	)
 	(global_label "PL_B35_L16_P"
 		(shape input)
@@
 		)
 	)
+	(global_label "MIO43"
+		(shape input)
+		(at 41.91 135.89 180)
+		(fields_autoplaced yes)
+		(effects
+			(font
+				(size 0.762 0.762)
+				(thickness 0.254)
+				(bold yes)
+			)
+			(justify right)
+		)
+		(property "Intersheetrefs" "${INTERSHEET_REFS}"
+			(at 36.1591 135.89 0)
+			(effects
+				(font
+					(size 1.27 1.27)
+				)
+				(justify right)
+				(hide yes)
+			)
+		)
+	)
 	(global_label "PL_B34_L7_P"
 		(shape input)
@@
 			(effects
 				(font
+					(size 1.27 1.27)
+				)
+				(justify right)
+				(hide yes)
+			)
+		)
+	)
+	(global_label "MIO45"
+		(shape input)
+		(at 41.91 128.27 180)
+		(fields_autoplaced yes)
+		(effects
+			(font
+				(size 0.762 0.762)
+				(thickness 0.254)
+				(bold yes)
+			)
+			(justify right)
+		)
+		(property "Intersheetrefs" "${INTERSHEET_REFS}"
+			(at 36.1591 128.27 0)
+			(effects
+				(font

Commit message: zynq_soc_complete_hdmi
Parts:
- removed J1001: 10144518-082802LF, Footprint-Lib-PhilsLab:10144518-082802LF, symbol Schematic-Lib-PhilsLab:10144518-082802LF
Connections:
- net PL_B35_L11_N: no longer names the net of J1000.41
- no-connect marks 4 -> 5
Other:
- note removed: "PL Bank 34 (DIFF)"
- moved on the sheet: J1000
