File: zynq_soc_board_v1.kicad_sch (KiCad schematic)
At the start: 1 part, among them U2 XC7Z020-2CLG400I

Commit message: sch-updated
Parts:
- removed unit 1 of U2
- removed unit 6 of U2

Commit message: sch_zynq_update
Parts:
- removed unit 4 of U2
- removed unit 3 of U2

Commit message: sch updated zynq ddr
Parts:
- removed U2: XC7Z020-2CLG400I, Package_BGA:Xilinx_CLG400, symbol 2024-11-30_12-42-37:XC7Z020-2CLG400I
Other:
- added sheet ethernet_gigabit (ethernet.kicad_sch)

Commit message: sch-eth-usb-updated
Other:
- added sheet Mezzanine_Connectors (Mezzanine Connectors.kicad_sch)
- added sheet USB-2-HS (USB-2-HS.kicad_sch)
Changed lines of the file:
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@@
+	)
+	(sheet
+		(at 207.01 142.24)
+		(size 69.85 17.78)
+		(fields_autoplaced yes)
+		(stroke
+			(width 0.1524)
+			(type solid)
+		)
+		(fill
+			(color 0 0 0 0.0000)
+		)
+		(property "Sheetname" "USB-2-HS"
+			(at 207.01 141.5284 0)
+			(effects
+				(font
+					(size 1.27 1.27)
+				)
+				(justify left bottom)
+			)
+		)
+		(property "Sheetfile" "USB-2-HS.kicad_sch"
+			(at 207.01 160.6046 0)
+			(effects
+				(font
+					(size 1.27 1.27)
+				)
+				(justify left top)
+			)
+		)
+		(instances
+			(project "zynq_soc_board_v1"
+				(path "/068a81e1-1783-4521-9958-788ddeed3b49"
+					(page "9")
+				)
+			)
+		)
 	)
 	(sheet
@@
 				)
 			)
+		)
+	)
+	(sheet
+		(at 120.65 172.72)
+		(size 49.53 19.05)
+		(fields_autoplaced yes)
+		(stroke
+			(width 0.1524)
+			(type solid)
+		)
+		(fill
+			(color 0 0 0 0.0000)
+		)
+		(property "Sheetname" "Mezzanine_Connectors"
+			(at 120.65 172.0084 0)
+			(effects
+				(font
+					(size 1.27 1.27)
+				)
+				(justify left bottom)
+			)
+		)
+		(property "Sheetfile" "Mezzanine Connectors.kicad_sch"
+			(at 120.65 192.3546 0)
+			(effects
+				(font
+					(size 1.27 1.27)
+				)
+				(justify left top)
+			)
+		)
+		(instances
+			(project "zynq_soc_board_v1"
+				(path "/068a81e1-1783-4521-9958-788ddeed3b49"
+					(page "10")
+				)
+			)

Commit message: zynq_soc_complete_hdmi
Other:
- added sheet hdmi (hdmi.kicad_sch)
Changed lines of the file:
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@@
+	)
+	(sheet
+		(at 118.11 40.64)
+		(size 68.58 34.29)
+		(fields_autoplaced yes)
+		(stroke
+			(width 0.1524)
+			(type solid)
+		)
+		(fill
+			(color 0 0 0 0.0000)
+		)
+		(property "Sheetname" "hdmi"
+			(at 118.11 39.9284 0)
+			(effects
+				(font
+					(size 1.27 1.27)
+				)
+				(justify left bottom)
+			)
+		)
+		(property "Sheetfile" "hdmi.kicad_sch"
+			(at 118.11 75.5146 0)
+			(effects
+				(font
+					(size 1.27 1.27)
+				)
+				(justify left top)
+			)
+		)
+		(instances
+			(project "zynq_soc_board_v1"
+				(path "/068a81e1-1783-4521-9958-788ddeed3b49"
+					(page "11")
+				)
+			)
+		)
 	)
 	(sheet
